File: Funkmodul1.sch (KiCad schematic (older format))
At the start: 44 parts

Commit message: Auto stash before merge of "master" and "github/master"
Parts:
- added D10: DZ2J036M0LCT-ND, Diodes_SMD:D_SOD-323F, symbol D_Zener
- added R15, R16, R17: 100k, Resistors_SMD:R_0603_HandSoldering, symbol R
- C10, C11, C12: renamed from C?; footprint Capacitors_SMD:C_0603 -> Capacitors_SMD:C_0603_HandSoldering
- C2: renamed from C?; footprint (none) -> Capacitors_SMD:C_1210_HandSoldering
- C5: renamed from C?; footprint (none) -> Capacitors_SMD:C_0603_HandSoldering
- Q1: renamed from Q?; footprint (none) -> TO_SOT_Packages_SMD:SOT-23
- Q2: renamed from Q?; value CSD13381F4 -> AO3414; footprint (none) -> TO_SOT_Packages_SMD:SOT-23
- U1: renamed from U?; footprint (none) -> Housings_SOIC:SOIC-16_3.9x9.9mm_Pitch1.27mm
- gave numbers to parts that had none: 35
Connections:
- net GND: now also D10.2 (A)
- net VCC: now also D10.1 (K), R15.1, R16.1, R17.1
- net TDI: now reaches U3.54 (PF7(ADC7/TDI))
- net TDI: now also R17.2
- net TDO: now reaches U3.55 (PF6(ADC6/TDO))
- net TMS: now reaches U3.56 (PF5(ADC5/TMS))
- net TMS: now also R16.2
- net TCK: now reaches U3.57 (PF4(ADC4/TCK))
- net TCK: now also R15.2
- net BAT_OK: now reaches U3.59 (PF2(ADC2))
Other:
- note added: "ESD Protection"
