File: Funkmodul1.sch (KiCad schematic (older format))
At the start: 47 parts, among them Q1 MMBT5401-TP, Q2 AO3414, U1 MC74HC4538A, U2 MAX892, U3 ATMEGA128-16AU, Y1 Crystal_GND23

Commit message: Adds Connectors
Parts:
- removed Y1: Crystal_GND23, Crystals:Crystal_SMD_EuroQuartz_X22-4pin_2.5x2.0mm_HandSoldering, symbol Crystal_GND23
- added C20: 100nF, Capacitors_SMD:C_0603_HandSoldering, symbol C
- added Y1: Crystal_GND24, Crystals:Crystal_SMD_3225-4pin_3.2x2.5mm_HandSoldering, symbol Crystal_GND24
Connections:
- wire segments 99 -> 101
Other:
- moved on the sheet: R4
Changed lines of the file:
@@
 LIBS:contrib
 LIBS:valves
+LIBS:nxp-ic
+LIBS:7400-ic
 LIBS:cubesatFunkmodul-cache
 LIBS:funkmodul
@@
 U 1 1 5993800E
 P 5250 1850
-F 0 "D?" H 5250 1950 50  0000 C CNN
+F 0 "D9" H 5250 1950 50  0000 C CNN
 F 1 "STTH102A" V 5050 2050 50  0000 C CNN
 F 2 "Diodes_SMD:D_0603" H 5250 1850 50  0001 C CNN
@@
 $EndComp
 Connection ~ 5250 2000
-$Comp
-L Crystal_GND23 Y1
-U 1 1 5993801C
-P 3750 2650
-F 0 "Y1" H 3875 2850 50  0000 L CNN
-F 1 "Crystal_GND23" H 3875 2775 50  0000 L CNN
-F 2 "Crystals:Crystal_SMD_EuroQuartz_X22-4pin_2.5x2.0mm_HandSoldering" H 3750 2650 50  0001 C CNN
-F 3 "" H 3750 2650 50  0001 C CNN
-	1    3750 2650
-	1    0    0    -1
-$EndComp
 Wire Wire Line
 	3900 2650 5200 2650
@@
 U 1 1 59B8D267
 P 2700 650
-F 0 "D?" H 2700 750 50  0000 C CNN
+F 0 "D4" H 2700 750 50  0000 C CNN
 F 1 "STTH102A" H 2700 550 50  0000 C CNN
 F 2 "Diodes_SMD:D_0603" H 2700 650 50  0001 C CNN
@@
 	0    1    1    0
 $EndComp
-Text HLabel 2700 2200 2    60   Input ~ 0
+Text HLabel 2800 2200 2    60   Input ~ 0
 3.3V
 Text HLabel 2500 3300 2    60   Input ~ 0
@@
 U 1 1 59C30428
 P 1000 1900
-F 0 "D?" H 1000 2000 50  0000 C CNN
+F 0 "D1" H 1000 2000 50  0000 C CNN
 F 1 "STTH102A" H 1000 1800 50  0000 C CNN
 F 2 "Diodes_SMD:D_0603" H 1000 1900 50  0001 C CNN
@@
 U 1 1 59C31C6C
 P 1150 2450
-F 0 "D?" H 1150 2550 50  0000 C CNN
+F 0 "D2" H 1150 2550 50  0000 C CNN
 F 1 "STTH102A" H 1150 2350 50  0000 C CNN
 F 2 "Diodes_SMD:D_0603" H 1150 2450 50  0001 C CNN
@@
 U 1 1 59C31DDE
 P 2850 2600
-F 0 "D?" H 2850 2700 50  0000 C CNN
+F 0 "D6" H 2850 2700 50  0000 C CNN
 F 1 "STTH102A" H 2700 2750 50  0000 C CNN
 F 2 "Diodes_SMD:D_0603" H 2850 2600 50  0001 C CNN
@@
 L R R4
 U 1 1 59C336BC
-P 1500 2100
-F 0 "R4" V 1580 2100 50  0000 C CNN
-F 1 "47R" V 1500 2100 50  0000 C CNN
-F 2 "Resistors_SMD:R_0603_HandSoldering" V 1430 2100 50  0001 C CNN
-F 3 "" H 1500 2100 50  0001 C CNN
-	1    1500 2100
-	0    1    1    0
-$EndComp
-Wire Wire Line
-	1300 2100 1350 2100
+P 1450 2100
+F 0 "R4" V 1530 2100 50  0000 C CNN
+F 1 "47R" V 1450 2100 50  0000 C CNN
+F 2 "Resistors_SMD:R_0603_HandSoldering" V 1380 2100 50  0001 C CNN
+F 3 "" H 1450 2100 50  0001 C CNN
+	1    1450 2100
+	0    1    1    0
+$EndComp
 Connection ~ 1300 1850
 Wire Wire Line
@@
 U 1 1 59C3CB02
 P 1200 2850
-F 0 "D?" H 1200 2950 50  0000 C CNN
+F 0 "D3" H 1200 2950 50  0000 C CNN
 F 1 "STTH102A" H 1200 2750 50  0000 C CNN
 F 2 "Diodes_SMD:D_0603" H 1200 2850 50  0001 C CNN
@@
 U 1 1 59C3D96E
 P 2850 1950
-F 0 "D?" H 2850 2050 50  0000 C CNN
+F 0 "D5" H 2850 2050 50  0000 C CNN
 F 1 "STTH102A " V 2950 2150 50  0000 C CNN
 F 2 "Diodes_SMD:D_0603" H 2850 1950 50  0001 C CNN
@@
 U 1 1 59C3FBB2
 P 3750 5400
-F 0 "D?" H 3750 5500 50  0000 C CNN
+F 0 "D8" H 3750 5500 50  0000 C CNN
 F 1 "STTH102A" V 3850 5250 50  0000 C CNN
 F 2 "Diodes_SMD:D_0603" H 3750 5400 50  0001 C CNN
@@
 U 1 1 59C3FB09
 P 3750 5000
-F 0 "D?" H 3750 5100 50  0000 C CNN
+F 0 "D7" H 3750 5100 50  0000 C CNN
 F 1 "STTH102A" V 3650 4900 50  0000 C CNN
 F 2 "Diodes_SMD:D_0603" H 3750 5000 50  0001 C CNN
@@
 Wire Wire Line
 	5100 4000 5550 4000
+Wire Wire Line
+	2700 2200 2800 2200
+Wire Wire Line
+	1600 2100 1650 2100
+$Comp
+L C C20
+U 1 1 59DB28E1
+P 1600 2250
+F 0 "C20" H 1625 2350 50  0000 L CNN
+F 1 "100nF" H 1625 2150 50  0000 L CNN
+F 2 "Capacitors_SMD:C_0603_HandSoldering" H 1638 2100 50  0001 C CNN
+F 3 "" H 1600 2250 50  0001 C CNN
+	1    1600 2250
+	1    0    0    -1
+$EndComp
+Connection ~ 1600 2100
+$Comp
+L GND #PWR027
+U 1 1 59DB2AE7
+P 1600 2400
+F 0 "#PWR027" H 1600 2150 50  0001 C CNN
+F 1 "GND" H 1600 2250 50  0000 C CNN
+F 2 "" H 1600 2400 50  0001 C CNN
+F 3 "" H 1600 2400 50  0001 C CNN
+	1    1600 2400
+	1    0    0    -1
+$EndComp
+$Comp
+L Crystal_GND24 Y1
+U 1 1 59DB4E21
+P 3750 2650
+F 0 "Y1" H 3875 2850 50  0000 L CNN
+F 1 "Crystal_GND24" H 3875 2775 50  0000 L CNN
+F 2 "Crystals:Crystal_SMD_3225-4pin_3.2x2.5mm_HandSoldering" H 3750 2650 50  0001 C CNN
+F 3 "" H 3750 2650 50  0001 C CNN
+	1    3750 2650
+	1    0    0    -1
+$EndComp
+Wire Wire Line
+	5550 4900 5250 4900
+Text Label 5250 4900 2    60   ~ 0
+BURNWIRE
 $EndSCHEMATC

Commit message: Layout Module1 prefinish
Modules Placed
Ground Plane placed
Supply Plane placed
TODO: Add cubesat connector, Place Antenna connector, Place burnwire connector, Review
Parts:
- D1, D2, D3, D4, D5, D6, D7, D8, D9: value STTH102A -> TS4148C
- U2: footprint (none) -> Maxim:µMAX-8
Connections:
- net labels removed: +3.3V
Changed lines of the file:
@@
 LIBS:contrib
 LIBS:valves
-LIBS:nxp-ic
-LIBS:7400-ic
 LIBS:cubesatFunkmodul-cache
 LIBS:funkmodul
-LIBS:DISCO_Connector
 EELAYER 25 0
 EELAYER END
@@
 P 5250 1850
 F 0 "D9" H 5250 1950 50  0000 C CNN
-F 1 "STTH102A" V 5050 2050 50  0000 C CNN
+F 1 "TS4148C" V 5050 2050 50  0000 C CNN
 F 2 "Diodes_SMD:D_0603" H 5250 1850 50  0001 C CNN
 F 3 "" H 5250 1850 50  0001 C CNN
@@
 F 0 "U2" H 2550 850 60  0000 C CNN
 F 1 "MAX892" H 2650 1550 60  0000 C CNN
-F 2 "" H 2550 850 60  0001 C CNN
+F 2 "Maxim:µMAX-8" H 2550 850 60  0001 C CNN
 F 3 "https://datasheets.maximintegrated.com/en/ds/MAX891L-MAX892L.pdf" H 2550 850 60  0001 C CNN
 	1    2700 1200
@@
 $EndComp
 $Comp
-L GND #PWR11
+L GND #PWR01
 U 1 1 59B7E482
 P 3200 1650
-F 0 "#PWR11" H 3200 1400 50  0001 C CNN
+F 0 "#PWR01" H 3200 1400 50  0001 C CNN
 F 1 "GND" H 3200 1500 50  0000 C CNN
 F 2 "" H 3200 1650 50  0001 C CNN
@@
 $EndComp
 $Comp
-L +3.3V #PWR12
-U 1 1 59B7E6D2
-P 3500 1250
-F 0 "#PWR12" H 3500 1100 50  0001 C CNN
-F 1 "+3.3V" H 3500 1390 50  0000 C CNN
-F 2 "" H 3500 1250 50  0001 C CNN
-F 3 "" H 3500 1250 50  0001 C CNN
-	1    3500 1250
-	0    1    1    0
-$EndComp
-$Comp
-L GND #PWR7
+L GND #PWR02
 U 1 1 59B7E738
 P 2250 1350
-F 0 "#PWR7" H 2250 1100 50  0001 C CNN
+F 0 "#PWR02" H 2250 1100 50  0001 C CNN
 F 1 "GND" H 2250 1200 50  0000 C CNN
 F 2 "" H 2250 1350 50  0001 C CNN
@@
 VCC
 $Comp
-L GND #PWR14
+L GND #PWR03
 U 1 1 59B80D24
 P 3750 2450
-F 0 "#PWR14" H 3750 2200 50  0001 C CNN
+F 0 "#PWR03" H 3750 2200 50  0001 C CNN
 F 1 "GND" H 3750 2300 50  0000 C CNN
 F 2 "" H 3750 2450 50  0001 C CNN
@@
 $EndComp
 $Comp
-L GND #PWR15
+L GND #PWR04
 U 1 1 59B80D8A
 P 3750 2850
-F 0 "#PWR15" H 3750 2600 50  0001 C CNN
+F 0 "#PWR04" H 3750 2600 50  0001 C CNN
 F 1 "GND" H 3750 2700 50  0000 C CNN
 F 2 "" H 3750 2850 50  0001 C CNN
@@
 $EndComp
 $Comp
-L GND #PWR18
+L GND #PWR05
 U 1 1 59B80E1B
 P 4300 3350
-F 0 "#PWR18" H 4300 3100 50  0001 C CNN
+F 0 "#PWR05" H 4300 3100 50  0001 C CNN
 F 1 "GND" H 4300 3200 50  0000 C CNN
 F 2 "" H 4300 3350 50  0001 C CNN
@@
 $EndComp
 $Comp
-L GND #PWR19
+L GND #PWR06
 U 1 1 59B80EAC
 P 4550 2350
-F 0 "#PWR19" H 4550 2100 50  0001 C CNN
+F 0 "#PWR06" H 4550 2100 50  0001 C CNN
 F 1 "GND" H 4550 2200 50  0000 C CNN
 F 2 "" H 4550 2350 50  0001 C CNN
@@
 $EndComp
 $Comp
-L GND #PWR20
+L GND #PWR07
 U 1 1 59B80F3D
 P 5000 2350
-F 0 "#PWR20" H 5000 2100 50  0001 C CNN
+F 0 "#PWR07" H 5000 2100 50  0001 C CNN
 F 1 "GND" H 5000 2200 50  0000 C CNN
 F 2 "" H 5000 2350 50  0001 C CNN
@@
 $EndComp
 $Comp
-L GND #PWR25
+L GND #PWR08
 U 1 1 59B835F0
 P 7000 1100
-F 0 "#PWR25" H 7000 850 50  0001 C CNN
+F 0 "#PWR08" H 7000 850 50  0001 C CNN
 F 1 "GND" H 7000 950 50  0000 C CNN
 F 2 "" H 7000 1100 50  0001 C CNN
@@
 $EndComp
 $Comp
-L GND #PWR22
+L GND #PWR09
 U 1 1 59B83656
 P 6500 1150
-F 0 "#PWR22" H 6500 900 50  0001 C CNN
+F 0 "#PWR09" H 6500 900 50  0001 C CNN
 F 1 "GND" H 6500 1000 50  0000 C CNN
 F 2 "" H 6500 1150 50  0001 C CNN
@@
 $EndComp
 $Comp
-L GND #PWR21
+L GND #PWR010
 U 1 1 59B836BC
 P 6200 1150
-F 0 "#PWR21" H 6200 900 50  0001 C CNN
+F 0 "#PWR010" H 6200 900 50  0001 C CNN
 F 1 "GND" H 6200 1000 50  0000 C CNN
 F 2 "" H 6200 1150 50  0001 C CNN
@@
 $EndComp
 $Comp
-L GND #PWR23
+L GND #PWR011
 U 1 1 59B847A7
 P 6600 5700
-F 0 "#PWR23" H 6600 5450 50  0001 C CNN
+F 0 "#PWR011" H 6600 5450 50  0001 C CNN
 F 1 "GND" H 6600 5550 50  0000 C CNN
 F 2 "" H 6600 5700 50  0001 C CNN
@@
 $EndComp
 $Comp
-L GND #PWR24
+L GND #PWR012
 U 1 1 59B8480D
 P 6700 5700
-F 0 "#PWR24" H 6700 5450 50  0001 C CNN
+F 0 "#PWR012" H 6700 5450 50  0001 C CNN
 F 1 "GND" H 6700 5550 50  0000 C CNN
 F 2 "" H 6700 5700 50  0001 C CNN
@@
 $EndComp
 $Comp
-L GND #PWR26
+L GND #PWR013
 U 1 1 59B84873
 P 7000 5700
-F 0 "#PWR26" H 7000 5450 50  0001 C CNN
+F 0 "#PWR013" H 7000 5450 50  0001 C CNN
 F 1 "GND" H 7000 5550 50  0000 C CNN
 F 2 "" H 7000 5700 50  0001 C CNN
@@
 	1650 2450 1650 2750
 $Comp
-L GND #PWR5
+L GND #PWR014
 U 1 1 59B8BFBA
 P 1650 2750
-F 0 "#PWR5" H 1650 2500 50  0001 C CNN
+F 0 "#PWR014" H 1650 2500 50  0001 C CNN
 F 1 "GND" H 1650 2600 50  0000 C CNN
 F 2 "" H 1650 2750 50  0001 C CNN
@@
 P 2700 650
 F 0 "D4" H 2700 750 50  0000 C CNN
-F 1 "STTH102A" H 2700 550 50  0000 C CNN
+F 1 "TS4148C" H 2700 550 50  0000 C CNN
 F 2 "Diodes_SMD:D_0603" H 2700 650 50  0001 C CNN
 F 3 "" H 2700 650 50  0001 C CNN
@@
 $EndComp
 $Comp
-L GND #PWR13
+L GND #PWR015
 U 1 1 59B8D4AD
 P 3600 750
-F 0 "#PWR13" H 3600 500 50  0001 C CNN
+F 0 "#PWR015" H 3600 500 50  0001 C CNN
 F 1 "GND" H 3600 600 50  0000 C CNN
 F 2 "" H 3600 750 50  0001 C CNN
@@
 $EndComp
 $Comp
-L GND #PWR6
+L GND #PWR016
 U 1 1 59B8D515
 P 1750 750
-F 0 "#PWR6" H 1750 500 50  0001 C CNN
+F 0 "#PWR016" H 1750 500 50  0001 C CNN
 F 1 "GND" H 1750 600 50  0000 C CNN
 F 2 "" H 1750 750 50  0001 C CNN
@@
 $EndComp
 $Comp
-L GND #PWR8
+L GND #PWR017
 U 1 1 59B94F70
 P 2650 4050
-F 0 "#PWR8" H 2650 3800 50  0001 C CNN
+F 0 "#PWR017" H 2650 3800 50  0001 C CNN
 F 1 "GND" H 2650 3900 50  0000 C CNN
 F 2 "" H 2650 4050 50  0001 C CNN
@@
 $EndComp
 $Comp
-L GND #PWR1
+L GND #PWR018
 U 1 1 59C3023F
 P 600 1500
-F 0 "#PWR1" H 600 1250 50  0001 C CNN
+F 0 "#PWR018" H 600 1250 50  0001 C CNN
 F 1 "GND" H 600 1350 50  0000 C CNN
 F 2 "" H 600 1500 50  0001 C CNN
@@
 P 1000 1900
 F 0 "D1" H 1000 2000 50  0000 C CNN
-F 1 "STTH102A" H 1000 1800 50  0000 C CNN
+F 1 "TS4148C" H 1000 1800 50  0000 C CNN
 F 2 "Diodes_SMD:D_0603" H 1000 1900 50  0001 C CNN
 F 3 "" H 1000 1900 50  0001 C CNN
@@
 P 1150 2450
 F 0 "D2" H 1150 2550 50  0000 C CNN
-F 1 "STTH102A" H 1150 2350 50  0000 C CNN
+F 1 "TS4148C" H 1150 2350 50  0000 C CNN
 F 2 "Diodes_SMD:D_0603" H 1150 2450 50  0001 C CNN
 F 3 "" H 1150 2450 50  0001 C CNN
@@
 P 2850 2600
 F 0 "D6" H 2850 2700 50  0000 C CNN
-F 1 "STTH102A" H 2700 2750 50  0000 C CNN
+F 1 "TS4148C" H 2700 2750 50  0000 C CNN
 F 2 "Diodes_SMD:D_0603" H 2850 2600 50  0001 C CNN
 F 3 "http://www.st.com/content/ccc/resource/technical/document/datasheet/98/bc/9f/6f/26/c3/4e/73/CD00002613.pdf/files/CD00002613.pdf/jcr:content/translations/en.CD00002613.pdf" H 2850 2600 50  0001 C CNN
@@
 $EndComp
 $Comp
-L GND #PWR2
+L GND #PWR019
 U 1 1 59C31F10
 P 800 4850
-F 0 "#PWR2" H 800 4600 50  0001 C CNN
+F 0 "#PWR019" H 800 4600 50  0001 C CNN
 F 1 "GND" H 800 4700 50  0000 C CNN
 F 2 "" H 800 4850 50  0001 C CNN
@@
 $EndComp
 $Comp
-L GND #PWR10
+L GND #PWR020
 U 1 1 59C39B79
 P 2950 3100
-F 0 "#PWR10" H 2950 2850 50  0001 C CNN
+F 0 "#PWR020" H 2950 2850 50  0001 C CNN
 F 1 "GND" H 2950 2950 50  0000 C CNN
 F 2 "" H 2950 3100 50  0001 C CNN
@@
 	1350 3000 1350 3100
 $Comp
-L GND #PWR3
+L GND #PWR021
 U 1 1 59C3C15C
 P 1350 3400
-F 0 "#PWR3" H 1350 3150 50  0001 C CNN
+F 0 "#PWR021" H 1350 3150 50  0001 C CNN
 F 1 "GND" H 1350 3250 50  0000 C CNN
 F 2 "" H 1350 3400 50  0001 C CNN
@@
 P 1200 2850
 F 0 "D3" H 1200 2950 50  0000 C CNN
-F 1 "STTH102A" H 1200 2750 50  0000 C CNN
+F 1 "TS4148C" H 1200 2750 50  0000 C CNN
 F 2 "Diodes_SMD:D_0603" H 1200 2850 50  0001 C CNN
 F 3 "" H 1200 2850 50  0001 C CNN
@@
 P 2850 1950
 F 0 "D5" H 2850 2050 50  0000 C CNN
-F 1 "STTH102A " V 2950 2150 50  0000 C CNN
+F 1 "TS4148C" V 2950 2150 50  0000 C CNN
 F 2 "Diodes_SMD:D_0603" H 2850 1950 50  0001 C CNN
 F 3 "http://www.st.com/content/ccc/resource/technical/document/datasheet/98/bc/9f/6f/26/c3/4e/73/CD00002613.pdf/files/CD00002613.pdf/jcr:content/translations/en.CD00002613.pdf" H 2850 1950 50  0001 C CNN
@@
 	2700 5750 2700 5600
 $Comp
-L GND #PWR9
+L GND #PWR022
 U 1 1 59C3F3E3
 P 2700 5750
-F 0 "#PWR9" H 2700 5500 50  0001 C CNN
+F 0 "#PWR022" H 2700 5500 50  0001 C CNN
 F 1 "GND" H 2700 5600 50  0000 C CNN
 F 2 "" H 2700 5750 50  0001 C CNN
@@
 $EndComp
 $Comp
-L GND #PWR16
+L GND #PWR023
 U 1 1 59C3FC57
 P 3750 5550
-F 0 "#PWR16" H 3750 5300 50  0001 C CNN
+F 0 "#PWR023" H 3750 5300 50  0001 C CNN
 F 1 "GND" H 3750 5400 50  0000 C CNN
 F 2 "" H 3750 5550 50  0001 C CNN
@@
 P 3750 5400
 F 0 "D8" H 3750 5500 50  0000 C CNN
-F 1 "STTH102A" V 3850 5250 50  0000 C CNN
+F 1 "TS4148C" V 3850 5250 50  0000 C CNN
 F 2 "Diodes_SMD:D_0603" H 3750 5400 50  0001 C CNN
 F 3 "" H 3750 5400 50  0001 C CNN
@@
 P 3750 5000
 F 0 "D7" H 3750 5100 50  0000 C CNN
-F 1 "STTH102A" V 3650 4900 50  0000 C CNN
+F 1 "TS4148C" V 3650 4900 50  0000 C CNN
 F 2 "Diodes_SMD:D_0603" H 3750 5000 50  0001 C CNN
 F 3 "" H 3750 5000 50  0001 C CNN
@@
 $EndComp
 $Comp
-L GND #PWR17
+L GND #PWR024
 U 1 1 59C4457A
 P 3950 5500
-F 0 "#PWR17" H 3950 5250 50  0001 C CNN
+F 0 "#PWR024" H 3950 5250 50  0001 C CNN
 F 1 "GND" H 3950 5350 50  0000 C CNN
 F 2 "" H 3950 5500 50  0001 C CNN
@@
 VCC
 $Comp
-L GND #PWR27
+L GND #PWR025
 U 1 1 59D3B876
 P 9100 1450
-F 0 "#PWR27" H 9100 1200 50  0001 C CNN
+F 0 "#PWR025" H 9100 1200 50  0001 C CNN
 F 1 "GND" H 9100 1300 50  0000 C CNN
 F 2 "" H 9100 1450 50  0001 C CNN
@@
 Connection ~ 1600 2100
 $Comp
-L GND #PWR4
+L GND #PWR026
 U 1 1 59DB2AE7
 P 1600 2400
-F 0 "#PWR4" H 1600 2150 50  0001 C CNN
+F 0 "#PWR026" H 1600 2150 50  0001 C CNN
 F 1 "GND" H 1600 2250 50  0000 C CNN
 F 2 "" H 1600 2400 50  0001 C CNN
@@
 Text Label 5250 4900 2    60   ~ 0
 BURNWIRE
+Text HLabel 3500 1250 2    60   Input ~ 0
+3.3V
 $EndSCHEMATC

Commit message: Replaces Q1 with p channel mosfet
Parts:
- removed Q1: MMBT5401-TP, TO_SOT_Packages_SMD:SOT-23, symbol Q_PNP_BCE
- added Q1: SSM3J334RLFTR-ND, TO_SOT_Packages_SMD:SOT-23, symbol Q_PMOS_DGS
Connections:
- net 3.3V: now also Q1.3 (S)
- net at D3.1 (K), D5.1 (K), R3.1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: now also Q1.1 (D)
- net at D1.1 (K), R1.1: now also Q1.2 (G)
Changed lines of the file:
@@
 $EndComp
 $Comp
-L GND #PWR11
+L GND #PWR01
 U 1 1 59B7E482
 P 3200 1650
-F 0 "#PWR11" H 3200 1400 50  0001 C CNN
+F 0 "#PWR01" H 3200 1400 50  0001 C CNN
 F 1 "GND" H 3200 1500 50  0000 C CNN
 F 2 "" H 3200 1650 50  0001 C CNN
@@
 $EndComp
 $Comp
-L GND #PWR7
+L GND #PWR02
 U 1 1 59B7E738
 P 2250 1350
-F 0 "#PWR7" H 2250 1100 50  0001 C CNN
+F 0 "#PWR02" H 2250 1100 50  0001 C CNN
 F 1 "GND" H 2250 1200 50  0000 C CNN
 F 2 "" H 2250 1350 50  0001 C CNN
@@
 VCC
 $Comp
-L GND #PWR13
+L GND #PWR03
 U 1 1 59B80D24
 P 3750 2450
-F 0 "#PWR13" H 3750 2200 50  0001 C CNN
+F 0 "#PWR03" H 3750 2200 50  0001 C CNN
 F 1 "GND" H 3750 2300 50  0000 C CNN
 F 2 "" H 3750 2450 50  0001 C CNN
@@
 $EndComp
 $Comp
-L GND #PWR14
+L GND #PWR04
 U 1 1 59B80D8A
 P 3750 2850
-F 0 "#PWR14" H 3750 2600 50  0001 C CNN
+F 0 "#PWR04" H 3750 2600 50  0001 C CNN
 F 1 "GND" H 3750 2700 50  0000 C CNN
 F 2 "" H 3750 2850 50  0001 C CNN
@@
 $EndComp
 $Comp
-L GND #PWR17
+L GND #PWR05
 U 1 1 59B80E1B
 P 4300 3350
-F 0 "#PWR17" H 4300 3100 50  0001 C CNN
+F 0 "#PWR05" H 4300 3100 50  0001 C CNN
 F 1 "GND" H 4300 3200 50  0000 C CNN
 F 2 "" H 4300 3350 50  0001 C CNN
@@
 $EndComp
 $Comp
-L GND #PWR18
+L GND #PWR06
 U 1 1 59B80EAC
 P 4550 2350
-F 0 "#PWR18" H 4550 2100 50  0001 C CNN
+F 0 "#PWR06" H 4550 2100 50  0001 C CNN
 F 1 "GND" H 4550 2200 50  0000 C CNN
 F 2 "" H 4550 2350 50  0001 C CNN
@@
 $EndComp
 $Comp
-L GND #PWR19
+L GND #PWR07
 U 1 1 59B80F3D
 P 5000 2350
-F 0 "#PWR19" H 5000 2100 50  0001 C CNN
+F 0 "#PWR07" H 5000 2100 50  0001 C CNN
 F 1 "GND" H 5000 2200 50  0000 C CNN
 F 2 "" H 5000 2350 50  0001 C CNN
@@
 $EndComp
 $Comp
-L GND #PWR24
+L GND #PWR08
 U 1 1 59B835F0
 P 7000 1100
-F 0 "#PWR24" H 7000 850 50  0001 C CNN
+F 0 "#PWR08" H 7000 850 50  0001 C CNN
 F 1 "GND" H 7000 950 50  0000 C CNN
 F 2 "" H 7000 1100 50  0001 C CNN
@@
 $EndComp
 $Comp
-L GND #PWR21
+L GND #PWR09
 U 1 1 59B83656
 P 6500 1150
-F 0 "#PWR21" H 6500 900 50  0001 C CNN
+F 0 "#PWR09" H 6500 900 50  0001 C CNN
 F 1 "GND" H 6500 1000 50  0000 C CNN
 F 2 "" H 6500 1150 50  0001 C CNN
@@
 $EndComp
 $Comp
-L GND #PWR20
+L GND #PWR010
 U 1 1 59B836BC
 P 6200 1150
-F 0 "#PWR20" H 6200 900 50  0001 C CNN
+F 0 "#PWR010" H 6200 900 50  0001 C CNN
 F 1 "GND" H 6200 1000 50  0000 C CNN
 F 2 "" H 6200 1150 50  0001 C CNN
@@
 $EndComp
 $Comp
-L GND #PWR22
+L GND #PWR011
 U 1 1 59B847A7
 P 6600 5700
-F 0 "#PWR22" H 6600 5450 50  0001 C CNN
+F 0 "#PWR011" H 6600 5450 50  0001 C CNN
 F 1 "GND" H 6600 5550 50  0000 C CNN
 F 2 "" H 6600 5700 50  0001 C CNN
@@
 $EndComp
 $Comp
-L GND #PWR23
+L GND #PWR012
 U 1 1 59B8480D
 P 6700 5700
-F 0 "#PWR23" H 6700 5450 50  0001 C CNN
+F 0 "#PWR012" H 6700 5450 50  0001 C CNN
 F 1 "GND" H 6700 5550 50  0000 C CNN
 F 2 "" H 6700 5700 50  0001 C CNN
@@
 $EndComp
 $Comp
-L GND #PWR25
+L GND #PWR013
 U 1 1 59B84873
 P 7000 5700
-F 0 "#PWR25" H 7000 5450 50  0001 C CNN
+F 0 "#PWR013" H 7000 5450 50  0001 C CNN
 F 1 "GND" H 7000 5550 50  0000 C CNN
 F 2 "" H 7000 5700 50  0001 C CNN
@@
 	1650 2450 1650 2750
 $Comp
-L GND #PWR5
+L GND #PWR014
 U 1 1 59B8BFBA
 P 1650 2750
-F 0 "#PWR5" H 1650 2500 50  0001 C CNN
+F 0 "#PWR014" H 1650 2500 50  0001 C CNN
 F 1 "GND" H 1650 2600 50  0000 C CNN
 F 2 "" H 1650 2750 50  0001 C CNN
@@
 $EndComp
 $Comp
-L GND #PWR12
+L GND #PWR015
 U 1 1 59B8D4AD
 P 3600 750
-F 0 "#PWR12" H 3600 500 50  0001 C CNN
+F 0 "#PWR015" H 3600 500 50  0001 C CNN
 F 1 "GND" H 3600 600 50  0000 C CNN
 F 2 "" H 3600 750 50  0001 C CNN
@@
 $EndComp
 $Comp
-L GND #PWR6
+L GND #PWR016
 U 1 1 59B8D515
 P 1750 750
-F 0 "#PWR6" H 1750 500 50  0001 C CNN
+F 0 "#PWR016" H 1750 500 50  0001 C CNN
 F 1 "GND" H 1750 600 50  0000 C CNN
 F 2 "" H 1750 750 50  0001 C CNN
@@
 $EndComp
 $Comp
-L GND #PWR8
+L GND #PWR017
 U 1 1 59B94F70
 P 2650 4050
-F 0 "#PWR8" H 2650 3800 50  0001 C CNN
+F 0 "#PWR017" H 2650 3800 50  0001 C CNN
 F 1 "GND" H 2650 3900 50  0000 C CNN
 F 2 "" H 2650 4050 50  0001 C CNN
@@
 $EndComp
 $Comp
-L GND #PWR1
+L GND #PWR018
 U 1 1 59C3023F
 P 600 1500
-F 0 "#PWR1" H 600 1250 50  0001 C CNN
+F 0 "#PWR018" H 600 1250 50  0001 C CNN
 F 1 "GND" H 600 1350 50  0000 C CNN
 F 2 "" H 600 1500 50  0001 C CNN
@@
 $EndComp
 $Comp
-L GND #PWR2
+L GND #PWR019
 U 1 1 59C31F10
 P 800 4850
-F 0 "#PWR2" H 800 4600 50  0001 C CNN
+F 0 "#PWR019" H 800 4600 50  0001 C CNN
 F 1 "GND" H 800 4700 50  0000 C CNN
 F 2 "" H 800 4850 50  0001 C CNN
@@
 Connection ~ 1000 1750
 $Comp
-L Q_PNP_BCE Q1
-U 1 1 59C37DB0
-P 1400 1500
-F 0 "Q1" H 1600 1550 50  0000 L CNN
-F 1 "MMBT5401-TP" H 1550 1350 50  0000 L CNN
-F 2 "TO_SOT_Packages_SMD:SOT-23" H 1600 1600 50  0001 C CNN
-F 3 "" H 1400 1500 50  0001 C CNN
-	1    1400 1500
-	-1   0    0    1
-$EndComp
-$Comp
 L C C4
 U 1 1 59C38D4B
@@
 $EndComp
 $Comp
-L GND #PWR10
+L GND #PWR020
 U 1 1 59C39B79
 P 2950 3100
-F 0 "#PWR10" H 2950 2850 50  0001 C CNN
+F 0 "#PWR020" H 2950 2850 50  0001 C CNN
 F 1 "GND" H 2950 2950 50  0000 C CNN
 F 2 "" H 2950 3100 50  0001 C CNN
@@
 	1350 3000 1350 3100
 $Comp
-L GND #PWR3
+L GND #PWR021
 U 1 1 59C3C15C
 P 1350 3400
-F 0 "#PWR3" H 1350 3150 50  0001 C CNN
+F 0 "#PWR021" H 1350 3150 50  0001 C CNN
 F 1 "GND" H 1350 3250 50  0000 C CNN
 F 2 "" H 1350 3400 50  0001 C CNN
@@
 	2700 5750 2700 5600
 $Comp
-L GND #PWR9
+L GND #PWR022
 U 1 1 59C3F3E3
 P 2700 5750
-F 0 "#PWR9" H 2700 5500 50  0001 C CNN
+F 0 "#PWR022" H 2700 5500 50  0001 C CNN
 F 1 "GND" H 2700 5600 50  0000 C CNN
 F 2 "" H 2700 5750 50  0001 C CNN
@@
 $EndComp
 $Comp
-L GND #PWR15
+L GND #PWR023
 U 1 1 59C3FC57
 P 3750 5550
-F 0 "#PWR15" H 3750 5300 50  0001 C CNN
+F 0 "#PWR023" H 3750 5300 50  0001 C CNN
 F 1 "GND" H 3750 5400 50  0000 C CNN
 F 2 "" H 3750 5550 50  0001 C CNN
@@
 $EndComp
 $Comp
-L GND #PWR16
+L GND #PWR024
 U 1 1 59C4457A
 P 3950 5500
-F 0 "#PWR16" H 3950 5250 50  0001 C CNN
+F 0 "#PWR024" H 3950 5250 50  0001 C CNN
 F 1 "GND" H 3950 5350 50  0000 C CNN
 F 2 "" H 3950 5500 50  0001 C CNN
@@
 VCC
 $Comp
-L GND #PWR26
+L GND #PWR025
 U 1 1 59D3B876
 P 9100 1450
-F 0 "#PWR26" H 9100 1200 50  0001 C CNN
+F 0 "#PWR025" H 9100 1200 50  0001 C CNN
 F 1 "GND" H 9100 1300 50  0000 C CNN
 F 2 "" H 9100 1450 50  0001 C CNN
@@
 Connection ~ 1600 2100
 $Comp
-L GND #PWR4
+L GND #PWR026
 U 1 1 59DB2AE7
 P 1600 2400
-F 0 "#PWR4" H 1600 2150 50  0001 C CNN
+F 0 "#PWR026" H 1600 2150 50  0001 C CNN
 F 1 "GND" H 1600 2250 50  0000 C CNN
 F 2 "" H 1600 2400 50  0001 C CNN
@@
 Text HLabel 3500 1250 2    60   Input ~ 0
 3.3V
+$Comp
+L Q_PMOS_DGS Q1
+U 1 1 59F0FE2A
+P 1400 1500
+F 0 "Q1" H 1600 1550 50  0000 L CNN
+F 1 "SSM3J334RLFTR-ND" H 1600 1350 50  0000 L CNN
+F 2 "TO_SOT_Packages_SMD:SOT-23" H 1600 1600 50  0001 C CNN
+F 3 "https://toshiba.semicon-storage.com/info/docget.jsp?did=5579&prodName=SSM3J334R" H 1400 1500 50  0001 C CNN
+	1    1400 1500
+	-1   0    0    1
+$EndComp
 $EndSCHEMATC
