File: Connector.sch (KiCad schematic (older format))
At the start: 7 parts

Commit message: Auto stash before merge of "master" and "github/master"
Parts:
- added CON1: SFML_TFML-120-STACK-CON1, DISCO_Connector_TFML_SFML-120-02-STACKED-A, symbol SFML_TFML-120-STACK-CON1
- added CON2: SFML_TFML-120-STACK-CON2, DISCO_Connector_TFML_SFML-120-02-STACKED-A, symbol SFML_TFML-120-STACK-CON2
- added D18: SMF3.3, symbol D_Zener
- D11, D12, D13, D14, D15, D16, D17: renamed from D?; value D_Zener -> SMF3.3
Connections:
- net GND: now also CON1.1 (GND), CON1.117 (GND), CON1.118 (GND), CON1.119 (GND), CON1.120 (GND), CON1.2 (GND), CON1.39 (GND), CON1.40 (GND), CON1.41 (GND), CON1.42 (GND), CON1.43 (GND), CON1.44 (GND), CON1.B1 (GND), CON1.B2 (GND), CON1.B39 (GND), CON1.B40 (GND), CON2.1 (GND), CON2.117 (GND), CON2.118 (GND), CON2.119 (GND), CON2.120 (GND), CON2.2 (GND), CON2.39 (GND), CON2.40 (GND), CON2.41 (GND), CON2.42 (GND), CON2.43 (GND), CON2.44 (GND), CON2.B1 (GND), CON2.B2 (GND), CON2.B39 (GND), CON2.B40 (GND), D18.2 (A)
- net RX1: now also CON2.23 (RADIO_RX), CON2.85 (RADIO_RX), CON2.86 (RADIO_RX), CON2.B18 (RADIO_RX)
- net RX2: now also CON2.24 (RADIO_RX), CON2.87 (RADIO_RX), CON2.88 (RADIO_RX), CON2.B17 (RADIO_RX)
- net TX1: now also CON2.21 (RADIO_TX), CON2.81 (RADIO_TX), CON2.82 (RADIO_TX), CON2.B20 (RADIO_TX)
- net TX2: now also CON2.22 (RADIO_TX), CON2.83 (RADIO_TX), CON2.84 (RADIO_TX), CON2.B19 (RADIO_TX)
- new net: CON1.10 (BAT1+), CON1.59 (BAT1+), CON1.60 (BAT1+), CON1.B31 (BAT1+)
- new net: CON1.100 (ISP_SCK), CON1.30 (ISP_SCK), CON1.99 (ISP_SCK), CON1.B11 (ISP_SCK)
- new net: CON1.101 (ISP_MISO), CON1.102 (ISP_MISO), CON1.31 (ISP_MISO), CON1.B10 (ISP_MISO)
- new net: CON1.103 (ISP_MISO), CON1.104 (ISP_MISO), CON1.32 (ISP_MISO), CON1.B9 (ISP_MISO)
- new net: CON1.105 (ISP_MOSI), CON1.106 (ISP_MOSI), CON1.33 (ISP_MOSI), CON1.B8 (ISP_MOSI)
- new net: CON1.107 (ISP_MOSI), CON1.108 (ISP_MOSI), CON1.34 (ISP_MOSI), CON1.B7 (ISP_MOSI)
- new net: CON1.109 (~ISP_RESET), CON1.110 (~ISP_RESET), CON1.35 (~ISP_RESET), CON1.B6 (~ISP_RESET)
- new net: CON1.11 (BAT1-), CON1.61 (BAT1-), CON1.62 (BAT1-), CON1.B30 (BAT1-)
- new net: CON1.111 (~ISP_RESET), CON1.112 (~ISP_RESET), CON1.36 (~ISP_RESET), CON1.B5 (~ISP_RESET)
- new net: CON1.113 (KS1), CON1.114 (KS1), CON1.37 (KS1), CON1.B4 (KS1)
- new net: CON1.115 (KS1), CON1.116 (KS1), CON1.38 (KS1), CON1.B3 (KS1)
- new net: CON1.12 (BAT1-), CON1.63 (BAT1-), CON1.64 (BAT1-), CON1.B29 (BAT1-)
- new net: CON1.13 (BAT2+), CON1.65 (BAT2+), CON1.66 (BAT2+), CON1.B28 (BAT2+)
- new net: CON1.14 (BAT2+), CON1.67 (BAT2+), CON1.68 (BAT2+), CON1.B27 (BAT2+)
- new net: CON1.15 (BAT2-), CON1.69 (BAT2-), CON1.70 (BAT2-), CON1.B26 (BAT2-)
- new net: CON1.16 (BAT2-), CON1.71 (BAT2-), CON1.72 (BAT2-), CON1.B25 (BAT2-)
- new net: CON1.17 (MT_RIN1), CON1.73 (MT_RIN1), CON1.74 (MT_RIN1), CON1.B24 (MT_RIN1)
- new net: CON1.18 (MT_RIN1), CON1.75 (MT_RIN1), CON1.76 (MT_RIN1), CON1.B23 (MT_RIN1)
- new net: CON1.19 (MT_FIN1), CON1.77 (MT_FIN1), CON1.78 (MT_FIN1), CON1.B22 (MT_FIN1)
- new net: CON1.20 (MT_FIN1), CON1.79 (MT_FIN1), CON1.80 (MT_FIN1), CON1.B21 (MT_FIN1)
- new net: CON1.21 (MT_RIN2), CON1.81 (MT_RIN2), CON1.82 (MT_RIN2), CON1.B20 (MT_RIN2)
- new net: CON1.22 (MT_RIN2), CON1.83 (MT_RIN2), CON1.84 (MT_RIN2), CON1.B19 (MT_RIN2)
- new net: CON1.23 (MT_FIN2), CON1.85 (MT_FIN2), CON1.86 (MT_FIN2), CON1.B18 (MT_FIN2)
- new net: CON1.24 (MT_FIN2), CON1.87 (MT_FIN2), CON1.88 (MT_FIN2), CON1.B17 (MT_FIN2)
- new net: CON1.25 (MT_RIN3), CON1.89 (MT_RIN3), CON1.90 (MT_RIN3), CON1.B16 (MT_RIN3)
- new net: CON1.26 (MT_RIN3), CON1.91 (MT_RIN3), CON1.92 (MT_RIN3), CON1.B15 (MT_RIN3)
- new net: CON1.27 (MT_FIN3), CON1.93 (MT_FIN3), CON1.94 (MT_FIN3), CON1.B14 (MT_FIN3)
- new net: CON1.28 (MT_FIN3), CON1.95 (MT_FIN3), CON1.96 (MT_FIN3), CON1.B13 (MT_FIN3)
- new net: CON1.29 (ISP_SCK), CON1.97 (ISP_SCK), CON1.98 (ISP_SCK), CON1.B12 (ISP_SCK)
- new net: CON1.53 (12V), CON1.54 (12V), CON1.7 (12V), CON1.B34 (12V)
- new net: CON1.55 (12V), CON1.56 (12V), CON1.8 (12V), CON1.B33 (12V)
- new net: CON1.57 (BAT1+), CON1.58 (BAT1+), CON1.9 (BAT1+), CON1.B32 (BAT1+)
- new net: CON2.10 (~SPI_CS), CON2.59 (~SPI_CS), CON2.60 (~SPI_CS), CON2.B31 (~SPI_CS)
- new net: CON2.100 (2), CON2.30 (2), CON2.99 (2), CON2.B11 (2)
- new net: CON2.101 (3), CON2.102 (3), CON2.31 (3), CON2.B10 (3)
- new net: CON2.103 (3), CON2.104 (3), CON2.32 (3), CON2.B9 (3)
- new net: CON2.105 (MT_EN), CON2.106 (MT_EN), CON2.33 (MT_EN), CON2.B8 (MT_EN)
- new net: CON2.107 (MT_EN), CON2.108 (MT_EN), CON2.34 (MT_EN), CON2.B7 (MT_EN)
- new net: CON2.109 (RBF), CON2.110 (RBF), CON2.35 (RBF), CON2.B6 (RBF)
- new net: CON2.11 (ADC_START), CON2.61 (ADC_START), CON2.62 (ADC_START), CON2.B30 (ADC_START)
- new net: CON2.111 (RBF), CON2.112 (RBF), CON2.36 (RBF), CON2.B5 (RBF)
- new net: CON2.113 (KS2), CON2.114 (KS2), CON2.37 (KS2), CON2.B4 (KS2)
- new net: CON2.115 (KS2), CON2.116 (KS2), CON2.38 (KS2), CON2.B3 (KS2)
- new net: CON2.12 (ADC_START), CON2.63 (ADC_START), CON2.64 (ADC_START), CON2.B29 (ADC_START)
- new net: CON2.13 (ADS_DR), CON2.65 (ADS_DR), CON2.66 (ADS_DR), CON2.B28 (ADS_DR)
- new net: CON2.14 (ADC_DR), CON2.67 (ADC_DR), CON2.68 (ADC_DR), CON2.B27 (ADC_DR)
- new net: CON2.17 (RS845_A), CON2.73 (RS845_A), CON2.74 (RS845_A), CON2.B24 (RS845_A)
- new net: CON2.18 (RS485_A), CON2.75 (RS485_A), CON2.76 (RS485_A), CON2.B23 (RS485_A)
- new net: CON2.19 (RS485_B), CON2.77 (RS485_B), CON2.78 (RS485_B), CON2.B22 (RS485_B)
- new net: CON2.20 (RS485_B), CON2.79 (RS485_B), CON2.80 (RS485_B), CON2.B21 (RS485_B)
- new net: CON2.25 (0), CON2.89 (0), CON2.90 (0), CON2.B16 (0)
- new net: CON2.26 (0), CON2.91 (0), CON2.92 (0), CON2.B15 (0)
- new net: CON2.27 (1), CON2.93 (1), CON2.94 (1), CON2.B14 (1)
- new net: CON2.28 (1), CON2.95 (1), CON2.96 (1), CON2.B13 (1)
- new net: CON2.29 (2), CON2.97 (2), CON2.98 (2), CON2.B12 (2)
- new net: CON2.3 (SPI_MISO), CON2.45 (SPI_MISO), CON2.46 (SPI_MISO), CON2.B38 (SPI_MISO)
- new net: CON2.4 (SPI_MISO), CON2.47 (SPI_MISO), CON2.48 (SPI_MISO), CON2.B37 (SPI_MISO)
- new net: CON2.49 (SPI_MOSI), CON2.5 (SPI_MOSI), CON2.50 (SPI_MOSI), CON2.B36 (SPI_MOSI)
- new net: CON2.51 (SPI_MOSI), CON2.52 (SPI_MOSI), CON2.6 (SPI_MOSI), CON2.B35 (SPI_MOSI)
- new net: CON2.53 (SPI_SCK), CON2.54 (SPI_SCK), CON2.7 (SPI_SCK), CON2.B34 (SPI_SCK)
- new net: CON2.55 (SPI_SCK), CON2.56 (SPI_SCK), CON2.8 (SPI_SCK), CON2.B33 (SPI_SCK)
- new net: CON2.57 (~SPI_CS), CON2.58 (~SPI_CS), CON2.9 (~SPI_CS), CON2.B32 (~SPI_CS)
- new net 3.3V: CON1.49 (3.3V), CON1.5 (3.3V), CON1.50 (3.3V), CON1.51 (3.3V), CON1.52 (3.3V), CON1.6 (3.3V), CON1.B35 (3.3V), CON1.B36 (3.3V)
- new net BAT_OK: CON2.15 (BAT_OK), CON2.16 (BAT_OK), CON2.69 (BAT_OK), CON2.70 (BAT_OK), CON2.71 (BAT_OK), CON2.72 (BAT_OK), CON2.B25 (BAT_OK), CON2.B26 (BAT_OK), D18.1 (K)
- new net VBAT: CON1.3 (PV-BUS), CON1.4 (PV_BUS), CON1.45 (PV-BUS), CON1.46 (PV-BUS), CON1.47 (PV_BUS), CON1.48 (PV_BUS), CON1.B37 (PV_BUS), CON1.B38 (PV-BUS)
Changed lines of the file:
@@
 LIBS:cubesatFunkmodul-cache
 LIBS:funkmodul
+LIBS:DISCO_Connector
 EELAYER 25 0
 EELAYER END
@@
 ~ENABLE1~
 $Comp
-L D_Zener D?
+L D_Zener D11
 U 1 1 59C451A8
 P 2300 4550
-F 0 "D?" H 2300 4650 50  0000 C CNN
-F 1 "D_Zener" H 2300 4450 50  0000 C CNN
+F 0 "D11" H 2300 4650 50  0000 C CNN
+F 1 "SMF3.3" H 2300 4450 50  0000 C CNN
 F 2 "" H 2300 4550 50  0001 C CNN
 F 3 "" H 2300 4550 50  0001 C CNN
@@
 $EndComp
 $Comp
-L D_Zener D?
+L D_Zener D12
 U 1 1 59C451CF
 P 2600 4550
-F 0 "D?" H 2600 4650 50  0000 C CNN
-F 1 "D_Zener" H 2600 4450 50  0000 C CNN
+F 0 "D12" H 2600 4650 50  0000 C CNN
+F 1 "SMF3.3" H 2600 4450 50  0000 C CNN
 F 2 "" H 2600 4550 50  0001 C CNN
 F 3 "" H 2600 4550 50  0001 C CNN
@@
 $EndComp
 $Comp
-L D_Zener D?
+L D_Zener D13
 U 1 1 59C451EA
 P 2900 4550
-F 0 "D?" H 2900 4650 50  0000 C CNN
-F 1 "D_Zener" H 2900 4450 50  0000 C CNN
+F 0 "D13" H 2900 4650 50  0000 C CNN
+F 1 "SMF3.3" H 2900 4450 50  0000 C CNN
 F 2 "" H 2900 4550 50  0001 C CNN
 F 3 "" H 2900 4550 50  0001 C CNN
@@
 $EndComp
 $Comp
-L GND #PWR?
+L GND #PWR037
 U 1 1 59C4523B
 P 2300 4700
-F 0 "#PWR?" H 2300 4450 50  0001 C CNN
+F 0 "#PWR037" H 2300 4450 50  0001 C CNN
 F 1 "GND" H 2300 4550 50  0000 C CNN
 F 2 "" H 2300 4700 50  0001 C CNN
@@
 $EndComp
 $Comp
-L GND #PWR?
+L GND #PWR038
 U 1 1 59C45255
 P 2600 4700
-F 0 "#PWR?" H 2600 4450 50  0001 C CNN
+F 0 "#PWR038" H 2600 4450 50  0001 C CNN
 F 1 "GND" H 2600 4550 50  0000 C CNN
 F 2 "" H 2600 4700 50  0001 C CNN
@@
 $EndComp
 $Comp
-L GND #PWR?
+L GND #PWR039
 U 1 1 59C4526F
 P 2900 4700
-F 0 "#PWR?" H 2900 4450 50  0001 C CNN
+F 0 "#PWR039" H 2900 4450 50  0001 C CNN
 F 1 "GND" H 2900 4550 50  0000 C CNN
 F 2 "" H 2900 4700 50  0001 C CNN
@@
 ~ENABLE2~
 $Comp
-L D_Zener D?
+L D_Zener D14
 U 1 1 59C452D2
 P 3400 4550
-F 0 "D?" H 3400 4650 50  0000 C CNN
-F 1 "D_Zener" H 3400 4450 50  0000 C CNN
+F 0 "D14" H 3400 4650 50  0000 C CNN
+F 1 "SMF3.3" H 3400 4450 50  0000 C CNN
 F 2 "" H 3400 4550 50  0001 C CNN
 F 3 "" H 3400 4550 50  0001 C CNN
@@
 $EndComp
 $Comp
-L D_Zener D?
+L D_Zener D15
 U 1 1 59C452D8
 P 3700 4550
-F 0 "D?" H 3700 4650 50  0000 C CNN
-F 1 "D_Zener" H 3700 4450 50  0000 C CNN
+F 0 "D15" H 3700 4650 50  0000 C CNN
+F 1 "SMF3.3" H 3700 4450 50  0000 C CNN
 F 2 "" H 3700 4550 50  0001 C CNN
 F 3 "" H 3700 4550 50  0001 C CNN
@@
 $EndComp
 $Comp
-L D_Zener D?
+L D_Zener D16
 U 1 1 59C452DE
 P 4000 4550
-F 0 "D?" H 4000 4650 50  0000 C CNN
-F 1 "D_Zener" H 4000 4450 50  0000 C CNN
+F 0 "D16" H 4000 4650 50  0000 C CNN
+F 1 "SMF3.3" H 4000 4450 50  0000 C CNN
 F 2 "" H 4000 4550 50  0001 C CNN
 F 3 "" H 4000 4550 50  0001 C CNN
@@
 $EndComp
 $Comp
-L GND #PWR?
+L GND #PWR040
 U 1 1 59C452E4
 P 3400 4700
-F 0 "#PWR?" H 3400 4450 50  0001 C CNN
+F 0 "#PWR040" H 3400 4450 50  0001 C CNN
 F 1 "GND" H 3400 4550 50  0000 C CNN
 F 2 "" H 3400 4700 50  0001 C CNN
@@
 $EndComp
 $Comp
-L GND #PWR?
+L GND #PWR041
 U 1 1 59C452EA
 P 3700 4700
-F 0 "#PWR?" H 3700 4450 50  0001 C CNN
+F 0 "#PWR041" H 3700 4450 50  0001 C CNN
 F 1 "GND" H 3700 4550 50  0000 C CNN
 F 2 "" H 3700 4700 50  0001 C CNN
@@
 $EndComp
 $Comp
-L GND #PWR?
+L GND #PWR042
 U 1 1 59C452F0
 P 4000 4700
-F 0 "#PWR?" H 4000 4450 50  0001 C CNN
+F 0 "#PWR042" H 4000 4450 50  0001 C CNN
 F 1 "GND" H 4000 4550 50  0000 C CNN
 F 2 "" H 4000 4700 50  0001 C CNN
@@
 WIRE_CONN
 $Comp
-L D_Zener D?
+L D_Zener D17
 U 1 1 59C45961
 P 4650 4550
-F 0 "D?" H 4650 4650 50  0000 C CNN
-F 1 "D_Zener" H 4650 4450 50  0000 C CNN
+F 0 "D17" H 4650 4650 50  0000 C CNN
+F 1 "SMF3.3" H 4650 4450 50  0000 C CNN
 F 2 "" H 4650 4550 50  0001 C CNN
 F 3 "" H 4650 4550 50  0001 C CNN
@@
 $EndComp
 $Comp
-L GND #PWR?
+L GND #PWR043
 U 1 1 59C45994
 P 4650 4700
-F 0 "#PWR?" H 4650 4450 50  0001 C CNN
+F 0 "#PWR043" H 4650 4450 50  0001 C CNN
 F 1 "GND" H 4650 4550 50  0000 C CNN
 F 2 "" H 4650 4700 50  0001 C CNN
@@
 Text Notes 3150 3800 0    60   ~ 0
 ESD Protection
+$Comp
+L SFML_TFML-120-STACK-CON1 CON1
+U 1 1 59DA7B1E
+P 2800 2200
+F 0 "CON1" H 2200 3320 45  0000 L BNN
+F 1 "SFML_TFML-120-STACK-CON1" H 2200 1120 45  0000 L BNN
+F 2 "DISCO_Connector_TFML_SFML-120-02-STACKED-A" H 2830 2350 20  0001 C CNN
+F 3 "" H 2800 2200 60  0001 C CNN
+	1    2800 2200
+	1    0    0    -1
+$EndComp
+$Comp
+L SFML_TFML-120-STACK-CON2 CON2
+U 1 1 59DA7C3F
+P 7050 2200
+F 0 "CON2" H 6450 3320 45  0000 L BNN
+F 1 "SFML_TFML-120-STACK-CON2" H 6450 1120 45  0000 L BNN
+F 2 "DISCO_Connector_TFML_SFML-120-02-STACKED-A" H 7080 2350 20  0001 C CNN
+F 3 "" H 7050 2200 60  0001 C CNN
+	1    7050 2200
+	1    0    0    -1
+$EndComp
+$Comp
+L GND #PWR044
+U 1 1 59DA7E4B
+P 7850 1200
+F 0 "#PWR044" H 7850 950 50  0001 C CNN
+F 1 "GND" H 7850 1050 50  0000 C CNN
+F 2 "" H 7850 1200 50  0001 C CNN
+F 3 "" H 7850 1200 50  0001 C CNN
+	1    7850 1200
+	0    -1   -1   0
+$EndComp
+$Comp
+L GND #PWR045
+U 1 1 59DA7E71
+P 6250 1200
+F 0 "#PWR045" H 6250 950 50  0001 C CNN
+F 1 "GND" H 6250 1050 50  0000 C CNN
+F 2 "" H 6250 1200 50  0001 C CNN
+F 3 "" H 6250 1200 50  0001 C CNN
+	1    6250 1200
+	0    1    1    0
+$EndComp
+$Comp
+L GND #PWR046
+U 1 1 59DA7F27
+P 6250 3100
+F 0 "#PWR046" H 6250 2850 50  0001 C CNN
+F 1 "GND" H 6250 2950 50  0000 C CNN
+F 2 "" H 6250 3100 50  0001 C CNN
+F 3 "" H 6250 3100 50  0001 C CNN
+	1    6250 3100
+	0    1    1    0
+$EndComp
+$Comp
+L GND #PWR047
+U 1 1 59DA7F4D
+P 7850 3100
+F 0 "#PWR047" H 7850 2850 50  0001 C CNN
+F 1 "GND" H 7850 2950 50  0000 C CNN
+F 2 "" H 7850 3100 50  0001 C CNN
+F 3 "" H 7850 3100 50  0001 C CNN
+	1    7850 3100
+	0    -1   -1   0
+$EndComp
+$Comp
+L GND #PWR048
+U 1 1 59DA801E
+P 3600 1200
+F 0 "#PWR048" H 3600 950 50  0001 C CNN
+F 1 "GND" H 3600 1050 50  0000 C CNN
+F 2 "" H 3600 1200 50  0001 C CNN
+F 3 "" H 3600 1200 50  0001 C CNN
+	1    3600 1200
+	0    -1   -1   0
+$EndComp
+$Comp
+L GND #PWR049
+U 1 1 59DA8044
+P 2000 1200
+F 0 "#PWR049" H 2000 950 50  0001 C CNN
+F 1 "GND" H 2000 1050 50  0000 C CNN
+F 2 "" H 2000 1200 50  0001 C CNN
+F 3 "" H 2000 1200 50  0001 C CNN
+	1    2000 1200
+	0    1    1    0
+$EndComp
+$Comp
+L GND #PWR050
+U 1 1 59DA8115
+P 2000 3100
+F 0 "#PWR050" H 2000 2850 50  0001 C CNN
+F 1 "GND" H 2000 2950 50  0000 C CNN
+F 2 "" H 2000 3100 50  0001 C CNN
+F 3 "" H 2000 3100 50  0001 C CNN
+	1    2000 3100
+	0    1    1    0
+$EndComp
+$Comp
+L GND #PWR051
+U 1 1 59DA82BE
+P 3600 3100
+F 0 "#PWR051" H 3600 2850 50  0001 C CNN
+F 1 "GND" H 3600 2950 50  0000 C CNN
+F 2 "" H 3600 3100 50  0001 C CNN
+F 3 "" H 3600 3100 50  0001 C CNN
+	1    3600 3100
+	0    -1   -1   0
+$EndComp
+Text HLabel 1650 1400 0    60   Input ~ 0
+3.3V
+Text HLabel 3850 1400 2    60   Input ~ 0
+3.3V
+Wire Wire Line
+	1650 1400 2000 1400
+Wire Wire Line
+	3600 1400 3850 1400
+Text GLabel 1650 1300 0    60   Input ~ 0
+VBAT
+Text GLabel 3900 1300 2    60   Input ~ 0
+VBAT
+Wire Wire Line
+	3600 1300 3900 1300
+Wire Wire Line
+	1650 1300 2000 1300
+Text HLabel 6250 2200 0    60   Input ~ 0
+TX1
+Text HLabel 6250 2300 0    60   Input ~ 0
+RX1
+Text HLabel 7850 2200 2    60   Input ~ 0
+TX2
+Text HLabel 7850 2300 2    60   Input ~ 0
+RX2
+Text HLabel 6250 1900 0    60   Input ~ 0
+BAT_OK
+Text HLabel 7850 1900 2    60   Input ~ 0
+BAT_OK
+Text HLabel 5100 4350 1    60   Input ~ 0
+BAT_OK
+$Comp
+L D_Zener D18
+U 1 1 59DAB8D7
+P 5100 4500
+F 0 "D18" H 5100 4600 50  0000 C CNN
+F 1 "SMF3.3" H 5100 4400 50  0000 C CNN
+F 2 "" H 5100 4500 50  0001 C CNN
+F 3 "" H 5100 4500 50  0001 C CNN
+	1    5100 4500
+	0    1    1    0
+$EndComp
+$Comp
+L GND #PWR052
+U 1 1 59DAB906
+P 5100 4650
+F 0 "#PWR052" H 5100 4400 50  0001 C CNN
+F 1 "GND" H 5100 4500 50  0000 C CNN
+F 2 "" H 5100 4650 50  0001 C CNN
+F 3 "" H 5100 4650 50  0001 C CNN
+	1    5100 4650
+	1    0    0    -1
+$EndComp
 $EndSCHEMATC

Commit message: Adds Connectors
Parts:
- D11, D12, D13, D14, D15, D16, D17, D18: footprint (none) -> Diodes_SMD:D_SOD-123F
Changed lines of the file:
@@
 LIBS:contrib
 LIBS:valves
+LIBS:nxp-ic
+LIBS:7400-ic
 LIBS:cubesatFunkmodul-cache
 LIBS:funkmodul
@@
 F 0 "D11" H 2300 4650 50  0000 C CNN
 F 1 "SMF3.3" H 2300 4450 50  0000 C CNN
-F 2 "" H 2300 4550 50  0001 C CNN
+F 2 "Diodes_SMD:D_SOD-123F" H 2300 4550 50  0001 C CNN
 F 3 "" H 2300 4550 50  0001 C CNN
 	1    2300 4550
@@
 F 0 "D12" H 2600 4650 50  0000 C CNN
 F 1 "SMF3.3" H 2600 4450 50  0000 C CNN
-F 2 "" H 2600 4550 50  0001 C CNN
+F 2 "Diodes_SMD:D_SOD-123F" H 2600 4550 50  0001 C CNN
 F 3 "" H 2600 4550 50  0001 C CNN
 	1    2600 4550
@@
 F 0 "D13" H 2900 4650 50  0000 C CNN
 F 1 "SMF3.3" H 2900 4450 50  0000 C CNN
-F 2 "" H 2900 4550 50  0001 C CNN
+F 2 "Diodes_SMD:D_SOD-123F" H 2900 4550 50  0001 C CNN
 F 3 "" H 2900 4550 50  0001 C CNN
 	1    2900 4550
@@
 $EndComp
 $Comp
-L GND #PWR037
+L GND #PWR038
 U 1 1 59C4523B
 P 2300 4700
-F 0 "#PWR037" H 2300 4450 50  0001 C CNN
+F 0 "#PWR038" H 2300 4450 50  0001 C CNN
 F 1 "GND" H 2300 4550 50  0000 C CNN
 F 2 "" H 2300 4700 50  0001 C CNN
@@
 $EndComp
 $Comp
-L GND #PWR038
+L GND #PWR039
 U 1 1 59C45255
 P 2600 4700
-F 0 "#PWR038" H 2600 4450 50  0001 C CNN
+F 0 "#PWR039" H 2600 4450 50  0001 C CNN
 F 1 "GND" H 2600 4550 50  0000 C CNN
 F 2 "" H 2600 4700 50  0001 C CNN
@@
 $EndComp
 $Comp
-L GND #PWR039
+L GND #PWR040
 U 1 1 59C4526F
 P 2900 4700
-F 0 "#PWR039" H 2900 4450 50  0001 C CNN
+F 0 "#PWR040" H 2900 4450 50  0001 C CNN
 F 1 "GND" H 2900 4550 50  0000 C CNN
 F 2 "" H 2900 4700 50  0001 C CNN
@@
 F 0 "D14" H 3400 4650 50  0000 C CNN
 F 1 "SMF3.3" H 3400 4450 50  0000 C CNN
-F 2 "" H 3400 4550 50  0001 C CNN
+F 2 "Diodes_SMD:D_SOD-123F" H 3400 4550 50  0001 C CNN
 F 3 "" H 3400 4550 50  0001 C CNN
 	1    3400 4550
@@
 F 0 "D15" H 3700 4650 50  0000 C CNN
 F 1 "SMF3.3" H 3700 4450 50  0000 C CNN
-F 2 "" H 3700 4550 50  0001 C CNN
+F 2 "Diodes_SMD:D_SOD-123F" H 3700 4550 50  0001 C CNN
 F 3 "" H 3700 4550 50  0001 C CNN
 	1    3700 4550
@@
 F 0 "D16" H 4000 4650 50  0000 C CNN
 F 1 "SMF3.3" H 4000 4450 50  0000 C CNN
-F 2 "" H 4000 4550 50  0001 C CNN
+F 2 "Diodes_SMD:D_SOD-123F" H 4000 4550 50  0001 C CNN
 F 3 "" H 4000 4550 50  0001 C CNN
 	1    4000 4550
@@
 $EndComp
 $Comp
-L GND #PWR040
+L GND #PWR041
 U 1 1 59C452E4
 P 3400 4700
-F 0 "#PWR040" H 3400 4450 50  0001 C CNN
+F 0 "#PWR041" H 3400 4450 50  0001 C CNN
 F 1 "GND" H 3400 4550 50  0000 C CNN
 F 2 "" H 3400 4700 50  0001 C CNN
@@
 $EndComp
 $Comp
-L GND #PWR041
+L GND #PWR042
 U 1 1 59C452EA
 P 3700 4700
-F 0 "#PWR041" H 3700 4450 50  0001 C CNN
+F 0 "#PWR042" H 3700 4450 50  0001 C CNN
 F 1 "GND" H 3700 4550 50  0000 C CNN
 F 2 "" H 3700 4700 50  0001 C CNN
@@
 $EndComp
 $Comp
-L GND #PWR042
+L GND #PWR043
 U 1 1 59C452F0
 P 4000 4700
-F 0 "#PWR042" H 4000 4450 50  0001 C CNN
+F 0 "#PWR043" H 4000 4450 50  0001 C CNN
 F 1 "GND" H 4000 4550 50  0000 C CNN
 F 2 "" H 4000 4700 50  0001 C CNN
@@
 F 0 "D17" H 4650 4650 50  0000 C CNN
 F 1 "SMF3.3" H 4650 4450 50  0000 C CNN
-F 2 "" H 4650 4550 50  0001 C CNN
+F 2 "Diodes_SMD:D_SOD-123F" H 4650 4550 50  0001 C CNN
 F 3 "" H 4650 4550 50  0001 C CNN
 	1    4650 4550
@@
 $EndComp
 $Comp
-L GND #PWR043
+L GND #PWR044
 U 1 1 59C45994
 P 4650 4700
-F 0 "#PWR043" H 4650 4450 50  0001 C CNN
+F 0 "#PWR044" H 4650 4450 50  0001 C CNN
 F 1 "GND" H 4650 4550 50  0000 C CNN
 F 2 "" H 4650 4700 50  0001 C CNN
@@
 $EndComp
 $Comp
-L GND #PWR044
+L GND #PWR045
 U 1 1 59DA7E4B
 P 7850 1200
-F 0 "#PWR044" H 7850 950 50  0001 C CNN
+F 0 "#PWR045" H 7850 950 50  0001 C CNN
 F 1 "GND" H 7850 1050 50  0000 C CNN
 F 2 "" H 7850 1200 50  0001 C CNN
@@
 $EndComp
 $Comp
-L GND #PWR045
+L GND #PWR046
 U 1 1 59DA7E71
 P 6250 1200
-F 0 "#PWR045" H 6250 950 50  0001 C CNN
+F 0 "#PWR046" H 6250 950 50  0001 C CNN
 F 1 "GND" H 6250 1050 50  0000 C CNN
 F 2 "" H 6250 1200 50  0001 C CNN
@@
 $EndComp
 $Comp
-L GND #PWR046
+L GND #PWR047
 U 1 1 59DA7F27
 P 6250 3100
-F 0 "#PWR046" H 6250 2850 50  0001 C CNN
+F 0 "#PWR047" H 6250 2850 50  0001 C CNN
 F 1 "GND" H 6250 2950 50  0000 C CNN
 F 2 "" H 6250 3100 50  0001 C CNN
@@
 $EndComp
 $Comp
-L GND #PWR047
+L GND #PWR048
 U 1 1 59DA7F4D
 P 7850 3100
-F 0 "#PWR047" H 7850 2850 50  0001 C CNN
+F 0 "#PWR048" H 7850 2850 50  0001 C CNN
 F 1 "GND" H 7850 2950 50  0000 C CNN
 F 2 "" H 7850 3100 50  0001 C CNN
@@
 $EndComp
 $Comp
-L GND #PWR048
+L GND #PWR049
 U 1 1 59DA801E
 P 3600 1200
-F 0 "#PWR048" H 3600 950 50  0001 C CNN
+F 0 "#PWR049" H 3600 950 50  0001 C CNN
 F 1 "GND" H 3600 1050 50  0000 C CNN
 F 2 "" H 3600 1200 50  0001 C CNN
@@
 $EndComp
 $Comp
-L GND #PWR049
+L GND #PWR050
 U 1 1 59DA8044
 P 2000 1200
-F 0 "#PWR049" H 2000 950 50  0001 C CNN
+F 0 "#PWR050" H 2000 950 50  0001 C CNN
 F 1 "GND" H 2000 1050 50  0000 C CNN
 F 2 "" H 2000 1200 50  0001 C CNN
@@
 $EndComp
 $Comp
-L GND #PWR050
+L GND #PWR051
 U 1 1 59DA8115
 P 2000 3100
-F 0 "#PWR050" H 2000 2850 50  0001 C CNN
+F 0 "#PWR051" H 2000 2850 50  0001 C CNN
 F 1 "GND" H 2000 2950 50  0000 C CNN
 F 2 "" H 2000 3100 50  0001 C CNN
@@
 $EndComp
 $Comp
-L GND #PWR051
+L GND #PWR052
 U 1 1 59DA82BE
 P 3600 3100
-F 0 "#PWR051" H 3600 2850 50  0001 C CNN
+F 0 "#PWR052" H 3600 2850 50  0001 C CNN
 F 1 "GND" H 3600 2950 50  0000 C CNN
 F 2 "" H 3600 3100 50  0001 C CNN
@@
 F 0 "D18" H 5100 4600 50  0000 C CNN
 F 1 "SMF3.3" H 5100 4400 50  0000 C CNN
-F 2 "" H 5100 4500 50  0001 C CNN
+F 2 "Diodes_SMD:D_SOD-123F" H 5100 4500 50  0001 C CNN
 F 3 "" H 5100 4500 50  0001 C CNN
 	1    5100 4500
@@
 $EndComp
 $Comp
-L GND #PWR052
+L GND #PWR053
 U 1 1 59DAB906
 P 5100 4650
-F 0 "#PWR052" H 5100 4400 50  0001 C CNN
+F 0 "#PWR053" H 5100 4400 50  0001 C CNN
 F 1 "GND" H 5100 4500 50  0000 C CNN
 F 2 "" H 5100 4650 50  0001 C CNN
