File: Connector.sch (KiCad schematic (older format))
At the start: 12 parts, among them CON11 DISCO-CON1, CON21 DISCO-CON2, J1 Conn_01x03

Commit message: Converted to new kicad version
Parts:
- CON11: symbol DISCO-CON1 -> cubesatFunkmodul-rescue:DISCO-CON1
- CON21: symbol DISCO-CON2 -> cubesatFunkmodul-rescue:DISCO-CON2
- D11, D12, D13, D14, D15, D16, D17, D18, D33: symbol D_Zener -> cubesatFunkmodul-rescue:D_Zener
- J1: symbol Conn_01x03 -> cubesatFunkmodul-rescue:Conn_01x03
Changed lines of the file:
@@
-EESchema Schematic File Version 2
-LIBS:power
-LIBS:device
-LIBS:transistors
-LIBS:conn
-LIBS:linear
-LIBS:regul
-LIBS:74xx
-LIBS:cmos4000
-LIBS:adc-dac
-LIBS:memory
-LIBS:xilinx
-LIBS:microcontrollers
-LIBS:dsp
-LIBS:microchip
-LIBS:analog_switches
-LIBS:motorola
-LIBS:texas
-LIBS:intel
-LIBS:audio
-LIBS:interface
-LIBS:digital-audio
-LIBS:philips
-LIBS:display
-LIBS:cypress
-LIBS:siliconi
-LIBS:opto
-LIBS:atmel
-LIBS:contrib
-LIBS:valves
-LIBS:nxp-ic
-LIBS:7400-ic
+EESchema Schematic File Version 4
 LIBS:cubesatFunkmodul-cache
-LIBS:funkmodul
-LIBS:CubeSat-Bus-1
-LIBS:CubeSat-Bus-2
-LIBS:disco-con
-LIBS:fiducial
-EELAYER 25 0
+EELAYER 26 0
 EELAYER END
 $Descr A4 11693 8268
@@
 ~ENABLE1~
 $Comp
-L D_Zener D11
+L cubesatFunkmodul-rescue:D_Zener D11
 U 1 1 59C451A8
 P 2300 4550
@@
 $EndComp
 $Comp
-L D_Zener D12
+L cubesatFunkmodul-rescue:D_Zener D12
 U 1 1 59C451CF
 P 2600 4550
@@
 $EndComp
 $Comp
-L D_Zener D13
+L cubesatFunkmodul-rescue:D_Zener D13
 U 1 1 59C451EA
 P 2900 4550
@@
 $EndComp
 $Comp
-L GND #PWR38
+L cubesatFunkmodul-rescue:GND #PWR38
 U 1 1 59C4523B
 P 2300 4700
@@
 $EndComp
 $Comp
-L GND #PWR39
+L cubesatFunkmodul-rescue:GND #PWR39
 U 1 1 59C45255
 P 2600 4700
@@
 $EndComp
 $Comp
-L GND #PWR40
+L cubesatFunkmodul-rescue:GND #PWR40
 U 1 1 59C4526F
 P 2900 4700
@@
 ~ENABLE2~
 $Comp
-L D_Zener D14
+L cubesatFunkmodul-rescue:D_Zener D14
 U 1 1 59C452D2
 P 3400 4550
@@
 $EndComp
 $Comp
-L D_Zener D15
+L cubesatFunkmodul-rescue:D_Zener D15
 U 1 1 59C452D8
 P 3700 4550
@@
 $EndComp
 $Comp
-L D_Zener D16
+L cubesatFunkmodul-rescue:D_Zener D16
 U 1 1 59C452DE
 P 4000 4550
@@
 $EndComp
 $Comp
-L GND #PWR41
+L cubesatFunkmodul-rescue:GND #PWR41
 U 1 1 59C452E4
 P 3400 4700
@@
 $EndComp
 $Comp
-L GND #PWR42
+L cubesatFunkmodul-rescue:GND #PWR42
 U 1 1 59C452EA
 P 3700 4700
@@
 $EndComp
 $Comp
-L GND #PWR43
+L cubesatFunkmodul-rescue:GND #PWR43
 U 1 1 59C452F0
 P 4000 4700
@@
 WIRE_CONN
 $Comp
-L D_Zener D17
+L cubesatFunkmodul-rescue:D_Zener D17
 U 1 1 59C45961
 P 4650 4550
@@
 $EndComp
 $Comp
-L GND #PWR44
+L cubesatFunkmodul-rescue:GND #PWR44
 U 1 1 59C45994
 P 4650 4700
@@
 ESD Protection
 $Comp
-L GND #PWR47
+L cubesatFunkmodul-rescue:GND #PWR47
 U 1 1 59DA7E71
 P 7100 1400
@@
 $EndComp
 $Comp
-L GND #PWR48
+L cubesatFunkmodul-rescue:GND #PWR48
 U 1 1 59DA7F27
 P 7100 4300
@@
 BAT_OK
 $Comp
-L D_Zener D18
+L cubesatFunkmodul-rescue:D_Zener D18
 U 1 1 59DAB8D7
 P 5100 4500
@@
 $EndComp
 $Comp
-L GND #PWR45
+L cubesatFunkmodul-rescue:GND #PWR45
 U 1 1 59DAB906
 P 5100 4650
@@
 $EndComp
 $Comp
-L DISCO-CON2 CON21
+L cubesatFunkmodul-rescue:DISCO-CON2 CON21
 U 1 1 59FBB064
 P 9950 2700
@@
 $EndComp
 $Comp
-L DISCO-CON1 CON11
+L cubesatFunkmodul-rescue:DISCO-CON1 CON11
 U 1 1 59FBB0E1
 P 6600 2800
@@
 ~RBF~
 $Comp
-L GND #PWR49
+L cubesatFunkmodul-rescue:GND #PWR49
 U 1 1 59FBC03F
 P 9450 1300
@@
 $EndComp
 $Comp
-L GND #PWR50
+L cubesatFunkmodul-rescue:GND #PWR50
 U 1 1 59FBC107
 P 9450 4300
@@
 WIRE_CONN2
 $Comp
-L D_Zener D33
+L cubesatFunkmodul-rescue:D_Zener D33
 U 1 1 5A0B499B
 P 5400 4550
@@
 $EndComp
 $Comp
-L GND #PWR46
+L cubesatFunkmodul-rescue:GND #PWR46
 U 1 1 5A0B49A1
 P 5400 4700
@@
 $EndComp
 $Comp
-L Conn_01x03 J1
+L cubesatFunkmodul-rescue:Conn_01x03 J1
 U 1 1 5A0DBE27
 P 6750 5100
