File: Funkeinheit.sch (KiCad schematic (older format))
At the start: 44 parts, among them Q3 MMBT5551-TP, Q4 MMBT5551-TP, Q5 MMBT5551-TP, Q6 MMBT5551-TP, Q7 MMBT5551-TP, Q8 MMBT5551-TP, U4 LTC3113, U5 RFM23BP

Commit message: Places µC of second module
Parts:
- Q3, Q4, Q5, Q6, Q7, Q8: symbol Q_NPN_BCE -> Q_NPN_BEC
Connections:
- net GND: now also Q8.2 (E); no longer Q8.3 (E)
- net MOSI: now also Q3.2 (E); no longer Q3.3 (E)
- net MOSI_: now also Q3.3 (C); no longer Q3.2 (C)
- net RXON: now also Q4.2 (E); no longer Q4.3 (E)
- net RXON_: now also Q4.3 (C); no longer Q4.2 (C)
- net SCK: now also Q7.2 (E); no longer Q7.3 (E)
- net SCK_: now also Q7.3 (C); no longer Q7.2 (C)
- net SS: now also Q6.2 (E); no longer Q6.3 (E)
- net SS_: now also Q6.3 (C); no longer Q6.2 (C)
- net TXON: now also Q5.2 (E); no longer Q5.3 (E)
- net TXON_: now also Q5.3 (C); no longer Q5.2 (C)
- net at R42.2, U4.14 (RUN): now also Q8.3 (C); no longer Q8.2 (C)
Changed lines of the file:
@@
 TXON
 $Comp
-L Q_NPN_BCE Q6
+L Q_NPN_BEC Q6
 U 1 1 59FF9D3E
 P 3600 1300
@@
 $EndComp
 $Comp
-L Q_NPN_BCE Q7
+L Q_NPN_BEC Q7
 U 1 1 599CAF76
 P 3600 1800
@@
 $EndComp
 $Comp
-L Q_NPN_BCE Q3
+L Q_NPN_BEC Q3
 U 1 1 599CAF95
 P 3550 2400
@@
 $EndComp
 $Comp
-L Q_NPN_BCE Q4
+L Q_NPN_BEC Q4
 U 1 1 599CB00B
 P 3550 2950
@@
 $EndComp
 $Comp
-L Q_NPN_BCE Q5
+L Q_NPN_BEC Q5
 U 1 1 599CB196
 P 3550 3450
@@
 	3800 1400 4250 1400
 $Comp
-L GND #PWR27
+L GND #PWR027
 U 1 1 59FF9D62
 P 3200 4450
-F 0 "#PWR27" H 3200 4200 50  0001 C CNN
+F 0 "#PWR027" H 3200 4200 50  0001 C CNN
 F 1 "GND" H 3200 4300 50  0000 C CNN
 F 2 "" H 3200 4450 50  0001 C CNN
@@
 $EndComp
 $Comp
-L GND #PWR29
+L GND #PWR028
 U 1 1 59FF9D63
 P 5750 3550
-F 0 "#PWR29" H 5750 3300 50  0001 C CNN
+F 0 "#PWR028" H 5750 3300 50  0001 C CNN
 F 1 "GND" H 5750 3400 50  0000 C CNN
 F 2 "" H 5750 3550 50  0001 C CNN
@@
 PGND
 $Comp
-L GND #PWR31
+L GND #PWR029
 U 1 1 59FF9D71
 P 7350 1900
-F 0 "#PWR31" H 7350 1650 50  0001 C CNN
+F 0 "#PWR029" H 7350 1650 50  0001 C CNN
 F 1 "GND" H 7350 1750 50  0000 C CNN
 F 2 "" H 7350 1900 50  0001 C CNN
@@
 5V
 $Comp
-L GND #PWR32
+L GND #PWR030
 U 1 1 59C59DAC
 P 7350 2000
-F 0 "#PWR32" H 7350 1750 50  0001 C CNN
+F 0 "#PWR030" H 7350 1750 50  0001 C CNN
 F 1 "GND" H 7350 1850 50  0000 C CNN
 F 2 "" H 7350 2000 50  0001 C CNN
@@
 	10550 1550 10550 1450
 $Comp
-L Q_NPN_BCE Q8
+L Q_NPN_BEC Q8
 U 1 1 59FF9D94
 P 10450 2100
@@
 	10550 1850 10550 1900
 $Comp
-L GND #PWR34
+L GND #PWR031
 U 1 1 59FF9D95
 P 10550 2300
-F 0 "#PWR34" H 10550 2050 50  0001 C CNN
+F 0 "#PWR031" H 10550 2050 50  0001 C CNN
 F 1 "GND" H 10550 2150 50  0000 C CNN
 F 2 "" H 10550 2300 50  0001 C CNN
@@
 $EndComp
 $Comp
-L GND #PWR30
+L GND #PWR032
 U 1 1 59FF9D98
 P 7050 2400
-F 0 "#PWR30" H 7050 2150 50  0001 C CNN
+F 0 "#PWR032" H 7050 2150 50  0001 C CNN
 F 1 "GND" H 7050 2250 50  0000 C CNN
 F 2 "" H 7050 2400 50  0001 C CNN
@@
 $EndComp
 $Comp
-L GND #PWR33
+L GND #PWR033
 U 1 1 59C6029F
 P 9750 2300
-F 0 "#PWR33" H 9750 2050 50  0001 C CNN
+F 0 "#PWR033" H 9750 2050 50  0001 C CNN
 F 1 "GND" H 9750 2150 50  0000 C CNN
 F 2 "" H 9750 2300 50  0001 C CNN
@@
 $EndComp
 $Comp
-L GND #PWR28
+L GND #PWR034
 U 1 1 59DE335D
 P 3200 5350
-F 0 "#PWR28" H 3200 5100 50  0001 C CNN
+F 0 "#PWR034" H 3200 5100 50  0001 C CNN
 F 1 "GND" H 3200 5200 50  0000 C CNN
 F 2 "" H 3200 5350 50  0001 C CNN

Commit message: Adds SMA and Burnwire connectors
Parts:
- AE1: footprint (none) -> Connectors:SMA_THT_Jack_Straight; symbol Antenna -> Antenna_Shield
Connections:
- net PGND: now also AE1.2 (Shield)
Changed lines of the file:
@@
 LIBS:contrib
 LIBS:valves
-LIBS:nxp-ic
-LIBS:7400-ic
 LIBS:cubesatFunkmodul-cache
 LIBS:funkmodul
-LIBS:CubeSat-Bus-1
-LIBS:CubeSat-Bus-2
 LIBS:disco-con
 EELAYER 25 0
@@
 5V
 $Comp
-L Antenna AE1
+L Antenna_Shield AE1
 U 1 1 59FF9DA2
 P 9700 3700
 F 0 "AE1" H 9625 3775 50  0000 R CNN
 F 1 "Antenna" H 9625 3700 50  0000 R CNN
-F 2 "" H 9700 3700 50  0001 C CNN
+F 2 "Connectors:SMA_THT_Jack_Straight" H 9700 3700 50  0001 C CNN
 F 3 "" H 9700 3700 50  0001 C CNN
 	1    9700 3700
@@
 3.3V to 5V Levelconverter
 Connection ~ 8400 5100
+Text Label 9800 3900 0    60   ~ 0
+PGND
 $EndSCHEMATC

Commit message: Adds stiching vias
Other:
- note added: "Precission resistors"
- note removed: "Precission resistors < 1%"
Changed lines of the file:
@@
 LIBS:contrib
 LIBS:valves
+LIBS:nxp-ic
+LIBS:7400-ic
 LIBS:cubesatFunkmodul-cache
 LIBS:funkmodul
+LIBS:CubeSat-Bus-1
+LIBS:CubeSat-Bus-2
 LIBS:disco-con
 EELAYER 25 0
@@
 	10250 1850 9650 1850
 Text Notes 9650 2800 0    60   ~ 0
-Precission resistors < 1%
+Precission resistors
 Text Label 9750 4450 0    60   ~ 0
 5V
