File: Funkeinheit2.sch (KiCad schematic (older format))
At the start: 44 parts, among them Q3 MMBT5551-TP, Q4 MMBT5551-TP, Q5 MMBT5551-TP, Q6 MMBT5551-TP, Q7 MMBT5551-TP, Q8 MMBT5551-TP, U4 LTC3113, U5 RFM23BP

Commit message: Adds new unit
Parts:
- removed AE1: Antenna, symbol Antenna
- removed C13, C14, C15: 47µF, Capacitors_SMD:C_1210_HandSoldering, symbol C
- removed C16: 47pF, Capacitors_SMD:C_0603_HandSoldering, symbol C
- removed C17: 680pF, Capacitors_SMD:C_0603_HandSoldering, symbol C
- removed C18: 12pF, Capacitors_SMD:C_0603_HandSoldering, symbol C
- removed C19: 100nF, Capacitors_SMD:C_0603_HandSoldering, symbol C
- removed L2: 5µH, Inductors_SMD:L_6.3x6.3_H3, symbol L
- removed Q3, Q4, Q5, Q6, Q7, Q8: MMBT5551-TP, TO_SOT_Packages_SMD:SOT-23, symbol Q_NPN_BCE
- removed R19, R21, R22, R23, R24, R25, R31, R32, R33, R34, R35, R41, R42, R44: 10k, Resistors_SMD:R_0603_HandSoldering, symbol R
- removed R20, R26, R27, R28, R29, R30, R45: 4k7, Resistors_SMD:R_0603_HandSoldering, symbol R
- removed R36: 90k9, Resistors_SMD:R_0603_HandSoldering, symbol R
- removed R37: 49k9, Resistors_SMD:R_0603_HandSoldering, symbol R
- removed R38: 6k81, Resistors_SMD:R_0603_HandSoldering, symbol R
- removed R39: 121k, Resistors_SMD:R_0603_HandSoldering, symbol R
- removed R40: 887k, Resistors_SMD:R_0603_HandSoldering, symbol R
- removed R43: 0R, Resistors_SMD:R_0603_HandSoldering, symbol R
- removed U4: LTC3113, Housings_SSOP:HTSSOP-20-1EP_4.4x6.5mm_Pitch0.65mm_ThermalPad, symbol LTC3113
- removed U5: RFM23BP, HopeRF:RFM23BP, symbol RFM23BP
- added AE2: Antenna, symbol Antenna
- added C34, C35, C36: 47µF, Capacitors_SMD:C_1210_HandSoldering, symbol C
- added C37: 47pF, Capacitors_SMD:C_0603_HandSoldering, symbol C
- added C38: 680pF, Capacitors_SMD:C_0603_HandSoldering, symbol C
- added C39: 12pF, Capacitors_SMD:C_0603_HandSoldering, symbol C
- added C40: 100nF, Capacitors_SMD:C_0603_HandSoldering, symbol C
- added L4: 5µH, Inductors_SMD:L_6.3x6.3_H3, symbol L
- added Q11, Q12, Q13, Q14, Q15, Q16: MMBT5551-TP, TO_SOT_Packages_SMD:SOT-23, symbol Q_NPN_BCE
- added R64, R65, R66, R67, R68, R69, R70, R78, R79, R80, R81, R82, R89, R90: 10k, Resistors_SMD:R_0603_HandSoldering, symbol R
- added R71, R72, R73, R74, R75, R76, R77: 4k7, Resistors_SMD:R_0603_HandSoldering, symbol R
- added R83: 0R, Resistors_SMD:R_0603_HandSoldering, symbol R
- added R84: 90k9, Resistors_SMD:R_0603_HandSoldering, symbol R
- added R85: 49k9, Resistors_SMD:R_0603_HandSoldering, symbol R
- added R86: 6k81, Resistors_SMD:R_0603_HandSoldering, symbol R
- added R87: 121k, Resistors_SMD:R_0603_HandSoldering, symbol R
- added R88: 887k, Resistors_SMD:R_0603_HandSoldering, symbol R
- added U10: RFM23BP, HopeRF:RFM23BP, symbol RFM23BP
- added U9: LTC3113, Housings_SSOP:HTSSOP-20-1EP_4.4x6.5mm_Pitch0.65mm_ThermalPad, symbol LTC3113
Connections:
- net +3.3V: now also R64.1, R65.1, R66.1, R67.1, R68.1, R71.2, R72.2, R73.2, R74.2, R75.2
- net 5V: now also C34.1, C35.1, C40.1, R78.1, R79.1, R80.1, R81.1, R82.1, R86.1, R88.1, U10.13 (VCC), U9.2 (VOUT), U9.3 (VOUT)
- net GND: now also Q16.3 (E), R69.2, R70.2, R83.2, R84.2, R87.2, U9.7 (SGND), U9.8 (BURST)
- net MISO: now also R69.1, R76.2
- net MISO_: now also R76.1, U10.2 (SDO)
- net MOSI: now also Q11.3 (E), R66.2
- net MOSI_: now also Q11.2 (C), R80.2, U10.3 (SDI)
- net NIRQ: now also R70.1, R77.2
- net NIRQ_: now also R77.1, U10.6 (NIRQ)
- net PGND: now also C34.2, C35.2, C36.2, C40.2, R83.1, U10.1 (GND), U10.10 (GND), U10.7 (SDN), U10.8 (GND), U9.1 (PGND), U9.10 (PGND), U9.11 (PGND), U9.20 (PGND), U9.21 (PAD)
- net RXON: now also Q12.3 (E), R67.2
- net RXON_: now also Q12.2 (C), R81.2, U10.12 (RXON)
- net SCK: now also Q15.3 (E), R65.2
- net SCK_: now also Q15.2 (C), R79.2, U10.4 (SCK)
- net SS: now also Q14.3 (E), R64.2
- net SS_: now also Q14.2 (C), R78.2, U10.5 (NSEL)
- net TXON: now also Q13.3 (E), R68.2
- net TXON_: now also Q13.2 (C), R82.2, U10.11 (TXON)
- net VBAT: now also C36.1, R90.1, U9.4 (VIN), U9.5 (VIN), U9.6 (VIN)
- net ~ENABLE~: now also R89.2
- new net: Q14.1 (B), R71.1
- new net: Q13.1 (B), R75.1
- new net: Q16.1 (B), R89.1
- new net: Q16.2 (C), R90.2, U9.14 (RUN)
- new net: R84.1, U9.9 (RT)
- new net: C37.1, R86.2
- new net: C37.2, C38.1, C39.1, R87.1, R88.2, U9.13 (FB)
- new net: C39.2, R85.2, U9.12 (VC)
- new net: AE2.1 (A), U10.9 (ANT)
- new net: C38.2, R85.1
- new net: Q15.1 (B), R72.1
- new net: Q11.1 (B), R73.1
- new net: Q12.1 (B), R74.1
- new net: L4.1, U9.18 (SW2), U9.19 (SW2)
- new net: L4.2, U9.15 (SW1), U9.16 (SW1), U9.17 (SW1)

Commit message: Places µC of second module
Parts:
- Q11, Q12, Q13, Q14, Q15, Q16: symbol Q_NPN_BCE -> Q_NPN_BEC
Connections:
- net GND: now also Q16.2 (E); no longer Q16.3 (E)
- net MOSI: now also Q11.2 (E); no longer Q11.3 (E)
- net MOSI_: now also Q11.3 (C); no longer Q11.2 (C)
- net RXON: now also Q12.2 (E); no longer Q12.3 (E)
- net RXON_: now also Q12.3 (C); no longer Q12.2 (C)
- net SCK: now also Q15.2 (E); no longer Q15.3 (E)
- net SCK_: now also Q15.3 (C); no longer Q15.2 (C)
- net SS: now also Q14.2 (E); no longer Q14.3 (E)
- net SS_: now also Q14.3 (C); no longer Q14.2 (C)
- net TXON: now also Q13.2 (E); no longer Q13.3 (E)
- net TXON_: now also Q13.3 (C); no longer Q13.2 (C)
- net at R90.2, U9.14 (RUN): now also Q16.3 (C); no longer Q16.2 (C)
Changed lines of the file:
@@
 TXON
 $Comp
-L Q_NPN_BCE Q?
+L Q_NPN_BEC Q?
 U 1 1 599CAE07
 P 3600 1300
@@
 $EndComp
 $Comp
-L Q_NPN_BCE Q?
+L Q_NPN_BEC Q?
 U 1 1 59FF9D3F
 P 3600 1800
@@
 $EndComp
 $Comp
-L Q_NPN_BCE Q?
+L Q_NPN_BEC Q?
 U 1 1 59FF9D40
 P 3550 2400
@@
 $EndComp
 $Comp
-L Q_NPN_BCE Q?
+L Q_NPN_BEC Q?
 U 1 1 59FF9D41
 P 3550 2950
@@
 $EndComp
 $Comp
-L Q_NPN_BCE Q?
+L Q_NPN_BEC Q?
 U 1 1 59FF9D42
 P 3550 3450
@@
 P 3200 4450
 AR Path="/59FF6F05/5994BAF1/59B87665" Ref="#PWR?"  Part="1"
-AR Path="/59FF6F05/59FF9D3B/59B87665" Ref="#PWR73"  Part="1"
-F 0 "#PWR73" H 3200 4200 50  0001 C CNN
+AR Path="/59FF6F05/59FF9D3B/59B87665" Ref="#PWR073"  Part="1"
+F 0 "#PWR073" H 3200 4200 50  0001 C CNN
 F 1 "GND" H 3200 4300 50  0000 C CNN
 F 2 "" H 3200 4450 50  0001 C CNN
@@
 P 5750 3550
 AR Path="/59FF6F05/5994BAF1/59B89289" Ref="#PWR?"  Part="1"
-AR Path="/59FF6F05/59FF9D3B/59B89289" Ref="#PWR75"  Part="1"
-F 0 "#PWR75" H 5750 3300 50  0001 C CNN
+AR Path="/59FF6F05/59FF9D3B/59B89289" Ref="#PWR074"  Part="1"
+F 0 "#PWR074" H 5750 3300 50  0001 C CNN
 F 1 "GND" H 5750 3400 50  0000 C CNN
 F 2 "" H 5750 3550 50  0001 C CNN
@@
 P 7350 1900
 AR Path="/59FF6F05/5994BAF1/59BD80CC" Ref="#PWR?"  Part="1"
-AR Path="/59FF6F05/59FF9D3B/59BD80CC" Ref="#PWR77"  Part="1"
-F 0 "#PWR77" H 7350 1650 50  0001 C CNN
+AR Path="/59FF6F05/59FF9D3B/59BD80CC" Ref="#PWR075"  Part="1"
+F 0 "#PWR075" H 7350 1650 50  0001 C CNN
 F 1 "GND" H 7350 1750 50  0000 C CNN
 F 2 "" H 7350 1900 50  0001 C CNN
@@
 P 7350 2000
 AR Path="/59FF6F05/5994BAF1/59FF9D92" Ref="#PWR?"  Part="1"
-AR Path="/59FF6F05/59FF9D3B/59FF9D92" Ref="#PWR78"  Part="1"
-F 0 "#PWR78" H 7350 1750 50  0001 C CNN
+AR Path="/59FF6F05/59FF9D3B/59FF9D92" Ref="#PWR076"  Part="1"
+F 0 "#PWR076" H 7350 1750 50  0001 C CNN
 F 1 "GND" H 7350 1850 50  0000 C CNN
 F 2 "" H 7350 2000 50  0001 C CNN
@@
 	10550 1550 10550 1450
 $Comp
-L Q_NPN_BCE Q?
+L Q_NPN_BEC Q?
 U 1 1 59C5A277
 P 10450 2100
@@
 P 10550 2300
 AR Path="/59FF6F05/5994BAF1/59C5A346" Ref="#PWR?"  Part="1"
-AR Path="/59FF6F05/59FF9D3B/59C5A346" Ref="#PWR80"  Part="1"
-F 0 "#PWR80" H 10550 2050 50  0001 C CNN
+AR Path="/59FF6F05/59FF9D3B/59C5A346" Ref="#PWR077"  Part="1"
+F 0 "#PWR077" H 10550 2050 50  0001 C CNN
 F 1 "GND" H 10550 2150 50  0000 C CNN
 F 2 "" H 10550 2300 50  0001 C CNN
@@
 P 7050 2400
 AR Path="/59FF6F05/5994BAF1/59C5FB2A" Ref="#PWR?"  Part="1"
-AR Path="/59FF6F05/59FF9D3B/59C5FB2A" Ref="#PWR76"  Part="1"
-F 0 "#PWR76" H 7050 2150 50  0001 C CNN
+AR Path="/59FF6F05/59FF9D3B/59C5FB2A" Ref="#PWR078"  Part="1"
+F 0 "#PWR078" H 7050 2150 50  0001 C CNN
 F 1 "GND" H 7050 2250 50  0000 C CNN
 F 2 "" H 7050 2400 50  0001 C CNN
@@
 P 9750 2300
 AR Path="/59FF6F05/5994BAF1/59FF9D9B" Ref="#PWR?"  Part="1"
-AR Path="/59FF6F05/59FF9D3B/59FF9D9B" Ref="#PWR79"  Part="1"
-F 0 "#PWR79" H 9750 2050 50  0001 C CNN
+AR Path="/59FF6F05/59FF9D3B/59FF9D9B" Ref="#PWR079"  Part="1"
+F 0 "#PWR079" H 9750 2050 50  0001 C CNN
 F 1 "GND" H 9750 2150 50  0000 C CNN
 F 2 "" H 9750 2300 50  0001 C CNN
@@
 P 3200 5350
 AR Path="/59FF6F05/5994BAF1/59FF9DAF" Ref="#PWR?"  Part="1"
-AR Path="/59FF6F05/59FF9D3B/59FF9DAF" Ref="#PWR74"  Part="1"
-F 0 "#PWR74" H 3200 5100 50  0001 C CNN
+AR Path="/59FF6F05/59FF9D3B/59FF9DAF" Ref="#PWR080"  Part="1"
+F 0 "#PWR080" H 3200 5100 50  0001 C CNN
 F 1 "GND" H 3200 5200 50  0000 C CNN
 F 2 "" H 3200 5350 50  0001 C CNN

Commit message: Adds SMA and Burnwire connectors
Parts:
- AE2: footprint (none) -> Connectors:SMA_THT_Jack_Straight; symbol Antenna -> Antenna_Shield
Connections:
- net PGND: now also AE2.2 (Shield)
Changed lines of the file:
@@
 LIBS:contrib
 LIBS:valves
-LIBS:nxp-ic
-LIBS:7400-ic
 LIBS:cubesatFunkmodul-cache
 LIBS:funkmodul
-LIBS:CubeSat-Bus-1
-LIBS:CubeSat-Bus-2
 LIBS:disco-con
 EELAYER 25 0
@@
 5V
 $Comp
-L Antenna AE?
+L Antenna_Shield AE?
 U 1 1 59C98C71
 P 9700 3700
@@
 F 0 "AE2" H 9625 3775 50  0000 R CNN
 F 1 "Antenna" H 9625 3700 50  0000 R CNN
-F 2 "" H 9700 3700 50  0001 C CNN
+F 2 "Connectors:SMA_THT_Jack_Straight" H 9700 3700 50  0001 C CNN
 F 3 "" H 9700 3700 50  0001 C CNN
 	1    9700 3700
@@
 3.3V to 5V Levelconverter
 Connection ~ 8400 5100
+Text Label 9800 3900 0    60   ~ 0
+PGND
 $EndSCHEMATC

Commit message: Adds stiching vias
Other:
- note added: "Precission resistors"
- note removed: "Precission resistors < 1%"
Changed lines of the file:
@@
 LIBS:contrib
 LIBS:valves
+LIBS:nxp-ic
+LIBS:7400-ic
 LIBS:cubesatFunkmodul-cache
 LIBS:funkmodul
+LIBS:CubeSat-Bus-1
+LIBS:CubeSat-Bus-2
 LIBS:disco-con
 EELAYER 25 0
@@
 	10250 1850 9650 1850
 Text Notes 9650 2800 0    60   ~ 0
-Precission resistors < 1%
+Precission resistors
 Text Label 9750 4450 0    60   ~ 0
 5V
