File: Funkeinheit2.sch (KiCad schematic (older format))
At the start: 44 parts, among them Q11 MMBT5551-TP, Q12 MMBT5551-TP, Q13 MMBT5551-TP, Q14 MMBT5551-TP, Q15 MMBT5551-TP, Q16 MMBT5551-TP, U10 RFM23BP, U9 LTC3113

Commit message: Converted to new kicad version
Parts:
- AE2: symbol Antenna_Shield -> cubesatFunkmodul-rescue:Antenna_Shield
- C34, C35, C36, C37, C38, C39, C40: symbol C -> cubesatFunkmodul-rescue:C
- L4: symbol L -> cubesatFunkmodul-rescue:L
- Q11, Q12, Q13, Q14, Q15, Q16: symbol Q_NPN_BEC -> cubesatFunkmodul-rescue:Q_NPN_BEC
- R64, R65, R66, R67, R68, R69, R70, R71, R72, R73, R74, R75, R76, R77, R78, R79, R80, R81, R82, R83, R84, R85, R86, R87, R88, R89, R90: symbol R -> cubesatFunkmodul-rescue:R
- U10: symbol RFM23BP -> cubesatFunkmodul-rescue:RFM23BP
- U9: symbol LTC3113 -> cubesatFunkmodul-rescue:LTC3113
Changed lines of the file:
@@
-EESchema Schematic File Version 2
-LIBS:power
-LIBS:device
-LIBS:transistors
-LIBS:conn
-LIBS:linear
-LIBS:regul
-LIBS:74xx
-LIBS:cmos4000
-LIBS:adc-dac
-LIBS:memory
-LIBS:xilinx
-LIBS:microcontrollers
-LIBS:dsp
-LIBS:microchip
-LIBS:analog_switches
-LIBS:motorola
-LIBS:texas
-LIBS:intel
-LIBS:audio
-LIBS:interface
-LIBS:digital-audio
-LIBS:philips
-LIBS:display
-LIBS:cypress
-LIBS:siliconi
-LIBS:opto
-LIBS:atmel
-LIBS:contrib
-LIBS:valves
-LIBS:nxp-ic
-LIBS:7400-ic
+EESchema Schematic File Version 4
 LIBS:cubesatFunkmodul-cache
-LIBS:funkmodul
-LIBS:CubeSat-Bus-1
-LIBS:CubeSat-Bus-2
-LIBS:disco-con
-LIBS:fiducial
-EELAYER 25 0
+EELAYER 26 0
 EELAYER END
 $Descr A4 11693 8268
@@
 MOSI_
 $Comp
-L R R?
+L cubesatFunkmodul-rescue:R R?
 U 1 1 59FF9D3C
 P 3200 4300
@@
 $EndComp
 $Comp
-L R R?
+L cubesatFunkmodul-rescue:R R?
 U 1 1 59FF9D3D
 P 3550 4100
@@
 TXON
 $Comp
-L Q_NPN_BEC Q?
+L cubesatFunkmodul-rescue:Q_NPN_BEC Q?
 U 1 1 599CAE07
 P 3600 1300
@@
 $EndComp
 $Comp
-L Q_NPN_BEC Q?
+L cubesatFunkmodul-rescue:Q_NPN_BEC Q?
 U 1 1 59FF9D3F
 P 3600 1800
@@
 $EndComp
 $Comp
-L Q_NPN_BEC Q?
+L cubesatFunkmodul-rescue:Q_NPN_BEC Q?
 U 1 1 59FF9D40
 P 3550 2400
@@
 $EndComp
 $Comp
-L Q_NPN_BEC Q?
+L cubesatFunkmodul-rescue:Q_NPN_BEC Q?
 U 1 1 59FF9D41
 P 3550 2950
@@
 $EndComp
 $Comp
-L Q_NPN_BEC Q?
+L cubesatFunkmodul-rescue:Q_NPN_BEC Q?
 U 1 1 59FF9D42
 P 3550 3450
@@
 $EndComp
 $Comp
-L R R?
+L cubesatFunkmodul-rescue:R R?
 U 1 1 599CB475
 P 3400 1000
@@
 $EndComp
 $Comp
-L R R?
+L cubesatFunkmodul-rescue:R R?
 U 1 1 59FF9D44
 P 3200 1250
@@
 $EndComp
 $Comp
-L R R?
+L cubesatFunkmodul-rescue:R R?
 U 1 1 59FF9D45
 P 3200 1750
@@
 $EndComp
 $Comp
-L R R?
+L cubesatFunkmodul-rescue:R R?
 U 1 1 59FF9D46
 P 3400 1550
@@
 $EndComp
 $Comp
-L R R?
+L cubesatFunkmodul-rescue:R R?
 U 1 1 59FF9D47
 P 3200 2350
@@
 $EndComp
 $Comp
-L R R?
+L cubesatFunkmodul-rescue:R R?
 U 1 1 59FF9D48
 P 3400 2150
@@
 $EndComp
 $Comp
-L R R?
+L cubesatFunkmodul-rescue:R R?
 U 1 1 599CB5CD
 P 3200 2900
@@
 $EndComp
 $Comp
-L R R?
+L cubesatFunkmodul-rescue:R R?
 U 1 1 59FF9D4A
 P 3400 2700
@@
 $EndComp
 $Comp
-L R R?
+L cubesatFunkmodul-rescue:R R?
 U 1 1 599CB649
 P 3200 3400
@@
 $EndComp
 $Comp
-L R R?
+L cubesatFunkmodul-rescue:R R?
 U 1 1 599CB6B7
 P 3400 3200
@@
 +3.3V
 $Comp
-L R R?
+L cubesatFunkmodul-rescue:R R?
 U 1 1 599CBEB7
 P 3900 1200
@@
 $EndComp
 $Comp
-L R R?
+L cubesatFunkmodul-rescue:R R?
 U 1 1 599CBEF0
 P 3900 1700
@@
 $EndComp
 $Comp
-L R R?
+L cubesatFunkmodul-rescue:R R?
 U 1 1 599CBF2D
 P 3900 2300
@@
 $EndComp
 $Comp
-L R R?
+L cubesatFunkmodul-rescue:R R?
 U 1 1 599CBF6A
 P 3900 2850
@@
 $EndComp
 $Comp
-L R R?
+L cubesatFunkmodul-rescue:R R?
 U 1 1 59FF9D51
 P 3900 3350
@@
 	3800 1400 4250 1400
 $Comp
-L GND #PWR?
+L cubesatFunkmodul-rescue:GND #PWR?
 U 1 1 59B87665
 P 3200 4450
@@
 $EndComp
 $Comp
-L GND #PWR?
+L cubesatFunkmodul-rescue:GND #PWR?
 U 1 1 59B89289
 P 5750 3550
@@
 PGND
 $Comp
-L GND #PWR?
+L cubesatFunkmodul-rescue:GND #PWR?
 U 1 1 59BD80CC
 P 7350 1900
@@
 	8600 1700 8950 1700
 $Comp
-L L L?
+L cubesatFunkmodul-rescue:L L?
 U 1 1 59FF9D72
 P 9100 1700
@@
 Connection ~ 7350 1450
 $Comp
-L C C?
+L cubesatFunkmodul-rescue:C C?
 U 1 1 59FF9D73
 P 6500 1600
@@
 $EndComp
 $Comp
-L C C?
+L cubesatFunkmodul-rescue:C C?
 U 1 1 59FF9D74
 P 6250 1600
@@
 Connection ~ 6500 1450
 $Comp
-L C C?
+L cubesatFunkmodul-rescue:C C?
 U 1 1 59FF9D75
 P 6900 1850
@@
 VBAT
 $Comp
-L LTC3113 U?
+L cubesatFunkmodul-rescue:LTC3113 U?
 U 1 1 59FF9D76
 P 8200 2050
@@
 5V
 $Comp
-L GND #PWR?
+L cubesatFunkmodul-rescue:GND #PWR?
 U 1 1 59FF9D92
 P 7350 2000
@@
 $EndComp
 $Comp
-L R R?
+L cubesatFunkmodul-rescue:R R?
 U 1 1 59FF9D93
 P 10550 1700
@@
 	10550 1550 10550 1450
 $Comp
-L Q_NPN_BEC Q?
+L cubesatFunkmodul-rescue:Q_NPN_BEC Q?
 U 1 1 59C5A277
 P 10450 2100
@@
 	10550 1850 10550 1900
 $Comp
-L GND #PWR?
+L cubesatFunkmodul-rescue:GND #PWR?
 U 1 1 59C5A346
 P 10550 2300
@@
 $EndComp
 $Comp
-L R R?
+L cubesatFunkmodul-rescue:R R?
 U 1 1 59C5A3D8
 P 10250 2250
@@
 	7350 2100 7050 2100
 $Comp
-L R R?
+L cubesatFunkmodul-rescue:R R?
 U 1 1 59C5FAC7
 P 7050 2250
@@
 $EndComp
 $Comp
-L GND #PWR?
+L cubesatFunkmodul-rescue:GND #PWR?
 U 1 1 59C5FB2A
 P 7050 2400
@@
 	8600 2000 9900 2000
 $Comp
-L R R?
+L cubesatFunkmodul-rescue:R R?
 U 1 1 59FF9D99
 P 10050 2000
@@
 $EndComp
 $Comp
-L R R?
+L cubesatFunkmodul-rescue:R R?
 U 1 1 59FF9D9A
 P 9750 2150
@@
 $EndComp
 $Comp
-L GND #PWR?
+L cubesatFunkmodul-rescue:GND #PWR?
 U 1 1 59FF9D9B
 P 9750 2300
@@
 5V
 $Comp
-L R R?
+L cubesatFunkmodul-rescue:R R?
 U 1 1 59C60B17
 P 9350 2100
@@
 $EndComp
 $Comp
-L C C?
+L cubesatFunkmodul-rescue:C C?
 U 1 1 59FF9D9D
 P 9050 2100
@@
 5V
 $Comp
-L C C?
+L cubesatFunkmodul-rescue:C C?
 U 1 1 59C60CFB
 P 9300 2500
@@
 $EndComp
 $Comp
-L R R?
+L cubesatFunkmodul-rescue:R R?
 U 1 1 59FF9D9F
 P 9050 2800
@@
 	6500 2000 6900 2000
 $Comp
-L RFM23BP U?
+L cubesatFunkmodul-rescue:RFM23BP U?
 U 1 1 59C696A7
 P 8500 4500
@@
 $EndComp
 $Comp
-L C C?
+L cubesatFunkmodul-rescue:C C?
 U 1 1 59C94242
 P 9050 2500
@@
 5V
 $Comp
-L Antenna_Shield AE?
+L cubesatFunkmodul-rescue:Antenna_Shield AE?
 U 1 1 59C98C71
 P 9700 3700
@@
 	9100 4450 9750 4450
 $Comp
-L C C?
+L cubesatFunkmodul-rescue:C C?
 U 1 1 59CB2ACF
 P 9600 4600
@@
 RXON_
 $Comp
-L R R?
+L cubesatFunkmodul-rescue:R R?
 U 1 1 59DBF7EA
 P 6150 3500
@@
 PGND
 $Comp
-L R R?
+L cubesatFunkmodul-rescue:R R?
 U 1 1 59DE3235
 P 3600 4950
@@
 $EndComp
 $Comp
-L R R?
+L cubesatFunkmodul-rescue:R R?
 U 1 1 59DE32B8
 P 3200 5200
@@
 $EndComp
 $Comp
-L GND #PWR?
+L cubesatFunkmodul-rescue:GND #PWR?
 U 1 1 59FF9DAF
 P 3200 5350
