File: cubesatFunkmodul.kicad_pcb (KiCad board)
At the start: 4 copper layers, 85 x 85 mm, 406 parts, among them CON11 DISCO-CON1, CON21 DISCO-CON2, J1 Conn_01x03, Q1 SSM3J334RLFTR-ND, Q10 AO3414, Q11 MMBT5551-TP, Q12 MMBT5551-TP, Q13 MMBT5551-TP, Q14 MMBT5551-TP, Q15 MMBT5551-TP, Q16 MMBT5551-TP, Q17 AO3414, Q18 AO3414, Q2 AO3414, Q3 MMBT5551-TP, Q4 MMBT5551-TP, Q5 MMBT5551-TP, Q6 MMBT5551-TP, Q7 MMBT5551-TP, Q8 MMBT5551-TP, Q9 SSM3J334RLFTR-ND, U1 MC74HC4538A, U10 RFM23BP, U2 MAX892, U3 ATMEGA128-16AU, U4 LTC3113, U5 RFM23BP, U6 MC74HC4538A, U7 MAX892, U8 ATMEGA128-16AU, U9 LTC3113, Y1 Crystal_GND24, Y2 Crystal_GND24

Commit message: Adds BOM and production files
Parts:
- removed the REF** at (74.6, 74.6)
- removed the REF** at (74.6, 73.9)
- added R15: 0R, Resistors_SMD:R_0805_HandSoldering, F.Cu at (58.9, 102.3)
- added R16: 0R, Resistors_SMD:R_0805_HandSoldering, B.Cu at (114.0, 106.5)
- Y1, Y2: value Crystal_GND24 -> 407F39D007M3728; footprint Crystals:Crystal_SMD_3225-4pin_3.2x2.5mm_HandSoldering -> Crystals:Crystal_SMD_7050-4pin_7.0x5.0mm
- moved C28 3.06 mm to (103.5, 101.6), turned to 270 degrees
- moved Y1 2.03 mm to (63.6, 96.9), turned to 0 degrees
- moved C29 1.44 mm to (99.7, 92.8)
- moved Y2 1.16 mm to (99.5, 97.9)
Connections:
- D24 pad 1: /Funkmodul2/~ON~ -> Net-(D24-Pad1)
- D6 pad 1: /Funkmodul1/~ON~ -> Net-(D6-Pad1)
- R51 pad 1: Net-(R51-Pad1) -> /Funkmodul2/~ON~
- R6 pad 1: Net-(R6-Pad1) -> /Funkmodul1/~ON~
- U1 pad 10: Net-(R6-Pad1) -> /Funkmodul1/~ON~
- U1 pad 5: Net-(R6-Pad1) -> /Funkmodul1/~ON~
- U3 pad 29: (no net) -> /Connector/3V3_Reset
- U6 pad 10: Net-(R51-Pad1) -> /Funkmodul2/~ON~
- U6 pad 5: Net-(R51-Pad1) -> /Funkmodul2/~ON~
- U8 pad 29: (no net) -> /Connector/3V3_Reset
Routing:
- net /Connector/3V3_Reset: track 0.00 -> 101.0 mm, vias 0 -> 2
- net /Funkmodul2/VCC: track 132.3 -> 154.9 mm
- net GND: track 716.0 -> 738.0 mm, vias 62 -> 67
- net Net-(R6-Pad1): track 18.0 -> 0.00 mm
- net /Funkmodul2/~ON~: track 69.1 -> 82.1 mm
- net /Funkmodul1/~ON~: track 86.7 -> 99.7 mm, vias 3 -> 2
- net /Funkmodul2/Funkeinheit2/PGND: track 61.5 -> 73.7 mm
- net VBAT: track 213.3 -> 224.7 mm
- net Net-(R51-Pad1): track 8.81 -> 0.00 mm
- net /Connector/TCK: track 99.8 -> 93.6 mm
- net Net-(C7-Pad1): track 8.01 -> 14.0 mm
- net Net-(CON11-Pad2): track 2.54 -> 6.68 mm
- net Net-(CON11-Pad29): track 2.54 -> 6.68 mm
- net Net-(CON21-Pad9): track 0.00 -> 3.81 mm
- net Net-(CON21-Pad8): track 0.00 -> 3.81 mm
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Other:
- net class Default: clearance 0.2032 -> 0.1524
- net class Supply: clearance 0.2032 -> 0.1524
- rule trace_clearance: 0.2032 -> 0.1524
- board text added: "ANT1"
- board text added: "ANT2"
- board text added: "Burnwire"
- board text added: "C1."
- board text added: "C2"
- board text added: "ID:"
- board text added: "TU WIEN SPACE TEAM RADIO V1.0"
- board text added: "VBAT/WIRE1/WIRE2"

Commit message: Adds via for shorter ground return path
Routing:
- net /Funkmodul1/Funkeinheit/PGND: track 47.2 -> 49.4 mm, vias 6 -> 7
Changed lines of the file:
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@@
     (links 1243)
     (no_connects 40)
-    (area 50.924999 33.924999 136.075001 119.075001)
+    (area 26.150001 32.4736 149.6245 138.700001)
     (thickness 1.6)
     (drawings 29)
-    (tracks 2109)
+    (tracks 2112)
     (zones 0)
     (modules 406)
@@
   )
   (setup
-    (last_trace_width 0.254)
+    (last_trace_width 0.2032)
     (user_trace_width 0.254)
     (user_trace_width 0.508)
@@
   (via (at 82.173321 93.785179) (size 0.6) (drill 0.3) (layers F.Cu B.Cu) (net 56))
   (segment (start 71.6559 98.5647) (end 71.5988 98.6218) (width 0.2032) (layer F.Cu) (net 56))
+  (segment (start 90.68716 73.43426) (end 90.68716 71.86014) (width 0.2032) (layer B.Cu) (net 57))
+  (segment (start 90.68716 71.86014) (end 91.1479 71.3994) (width 0.2032) (layer B.Cu) (net 57))
+  (via (at 91.1479 71.3994) (size 0.6) (drill 0.3) (layers F.Cu B.Cu) (net 57))
   (segment (start 91.0463 77.6097) (end 91.0463 74.9747) (width 1.016) (layer In2.Cu) (net 57))
   (segment (start 96.1263 82.6897) (end 96.1263 77.6097) (width 1.016) (layer In2.Cu) (net 57))

Commit message: Closes Ground Ring
Routing:
- net GND: track 738.0 -> 866.5 mm
Changed lines of the file:
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@@
     (thickness 1.6)
     (drawings 29)
-    (tracks 2112)
+    (tracks 2134)
     (zones 0)
     (modules 406)
@@
   (segment (start 59.9126 71.0819) (end 59.9126 70.0719) (width 0.254) (layer F.Cu) (net 9))
   (segment (start 59.9126 70.0719) (end 59.9186 70.0659) (width 0.254) (layer F.Cu) (net 9))
+  (segment (start 51.689 53.152) (end 52.0641 53.152) (width 0.508) (layer F.Cu) (net 10))
+  (segment (start 52.0641 53.152) (end 52.468 53.5559) (width 0.508) (layer F.Cu) (net 10))
+  (segment (start 51.689 51.417) (end 51.689 53.152) (width 0.508) (layer F.Cu) (net 10))
+  (segment (start 51.689 47.2305) (end 51.689 51.417) (width 0.508) (layer In2.Cu) (net 10))
+  (segment (start 51.689 40.95075) (end 51.689 47.2305) (width 0.508) (layer In2.Cu) (net 10))
+  (segment (start 51.689 34.671) (end 51.689 40.95075) (width 0.508) (layer In2.Cu) (net 10))
+  (segment (start 135.419 45.13725) (end 135.419 51.417) (width 0.508) (layer In2.Cu) (net 10))
+  (segment (start 135.419 38.8575) (end 135.419 45.13725) (width 0.508) (layer In2.Cu) (net 10))
+  (segment (start 135.419 34.671) (end 135.419 38.8575) (width 0.508) (layer In2.Cu) (net 10))
+  (segment (start 51.689 53.082) (end 52.1629 53.5559) (width 0.508) (layer B.Cu) (net 10))
+  (segment (start 52.1629 53.5559) (end 52.47161 53.5559) (width 0.508) (layer B.Cu) (net 10))
+  (segment (start 51.689 51.417) (end 51.689 53.082) (width 0.508) (layer B.Cu) (net 10))
+  (segment (start 135.419 34.671) (end 131.2325 34.671) (width 0.508) (layer B.Cu) (net 10))
+  (segment (start 122.8595 34.671) (end 131.2325 34.671) (width 0.508) (layer B.Cu) (net 10))
+  (segment (start 122.8595 34.671) (end 135.419 34.671) (width 0.508) (layer F.Cu) (net 10))
+  (segment (start 51.689 34.671) (end 51.689 51.417) (width 0.508) (layer B.Cu) (net 10))
+  (segment (start 68.435 34.671) (end 68.010736 34.671) (width 0.508) (layer B.Cu) (net 10))
+  (segment (start 68.010736 34.671) (end 51.689 34.671) (width 0.508) (layer B.Cu) (net 10))
+  (segment (start 114.4865 34.671) (end 68.435 34.671) (width 0.508) (layer B.Cu) (net 10))
+  (segment (start 135.419 93.282) (end 135.419 91.5269) (width 0.508) (layer F.Cu) (net 10))
+  (segment (start 135.419 91.5269) (end 134.278 90.3859) (width 0.508) (layer F.Cu) (net 10))
+  (segment (start 135.419 51.417) (end 135.419 52.4149) (width 0.508) (layer F.Cu) (net 10))
+  (segment (start 135.419 52.4149) (end 134.278 53.5559) (width 0.508) (layer F.Cu) (net 10))
+  (segment (start 135.419 34.671) (end 135.419 51.417) (width 0.508) (layer F.Cu) (net 10))
+  (segment (start 114.4865 34.671) (end 122.8595 34.671) (width 0.508) (layer F.Cu) (net 10))
   (segment (start 52.468 53.5559) (end 53.748666 53.5559) (width 0.508) (layer F.Cu) (net 10))
   (segment (start 53.748666 53.5559) (end 54.148665 53.155901) (width 0.508) (layer F.Cu) (net 10))
@@
   (segment (start 135.419 51.417) (end 135.419 51.841264) (width 0.508) (layer In2.Cu) (net 10))
   (segment (start 135.419 51.841264) (end 135.4145 51.845764) (width 0.508) (layer In2.Cu) (net 10))
-  (segment (start 135.419 34.671) (end 135.419 51.417) (width 0.508) (layer In2.Cu) (net 10))
   (segment (start 51.689 34.671) (end 86.301658 34.671) (width 0.508) (layer In2.Cu) (net 10))
   (segment (start 86.301658 34.671) (end 135.419 34.671) (width 0.508) (layer In2.Cu) (net 10))
-  (segment (start 51.689 51.417) (end 51.689 34.671) (width 0.508) (layer In2.Cu) (net 10))
   (segment (start 51.6945 51.846764) (end 51.6945 52.9518) (width 0.508) (layer In2.Cu) (net 10))
   (segment (start 51.6945 52.9518) (end 52.2986 53.5559) (width 0.508) (layer In2.Cu) (net 10))
   (segment (start 51.689 51.417) (end 51.689 51.841264) (width 0.508) (layer In2.Cu) (net 10))
   (segment (start 51.689 51.841264) (end 51.6945 51.846764) (width 0.508) (layer In2.Cu) (net 10))
-  (segment (start 122.8595 34.671) (end 135.419 34.671) (width 0.508) (layer F.Cu) (net 10))
   (segment (start 51.689 34.671) (end 52.113264 34.671) (width 0.508) (layer F.Cu) (net 10))
   (segment (start 52.113264 34.671) (end 114.4865 34.671) (width 0.508) (layer F.Cu) (net 10))

Commit message: Adds Coordinatesystem and bom selection
Parts:
- added G***: LOGO, Logos:Coordinate, F.Cu at (128.6, 41.0)
Changed lines of the file:
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@@
 (kicad_pcb (version 4) (host pcbnew 4.0.6)
   (general
-    (links 1243)
+    (links 0)
     (no_connects 40)
     (area 26.150001 32.4736 149.6245 138.700001)
@@
     (tracks 2134)
     (zones 0)
-    (modules 406)
+    (modules 407)
     (nets 175)
   )
@@
     (35 F.Paste user hide)
     (36 B.SilkS user hide)
-    (37 F.SilkS user hide)
+    (37 F.SilkS user)
     (38 B.Mask user hide)
     (39 F.Mask user hide)
@@
     )
   )
+  (module Logos:Coordinate (layer F.Cu)
+    (at 128.5645 41.0265)
+    (fp_text reference G*** (at 0 0) (layer F.SilkS) hide
+      (effects (font (thickness 0.3)))
+    )
+    (fp_text value LOGO (at 0.75 0) (layer F.SilkS) hide
+      (effects (font (thickness 0.3)))
+    )
+    (fp_poly (pts (xy -4.058272 3.452969) (xy -4.004048 3.529816) (xy -4.057972 3.666942) (xy -4.1275 3.763827)
+      (xy -4.227925 3.904527) (xy -4.238712 3.975265) (xy -4.15678 3.999011) (xy -4.09575 4.0005)
+      (xy -3.976414 4.022236) (xy -3.937 4.064) (xy -3.993335 4.103763) (xy -4.134064 4.12588)
+      (xy -4.191 4.1275) (xy -4.350042 4.112479) (xy -4.438515 4.074956) (xy -4.445 4.059763)
+      (xy -4.409174 3.970913) (xy -4.319367 3.829372) (xy -4.278714 3.774013) (xy -4.112427 3.556)
+      (xy -4.278714 3.556) (xy -4.401609 3.535163) (xy -4.445 3.4925) (xy -4.389179 3.450528)
+      (xy -4.251918 3.429548) (xy -4.22275 3.429) (xy -4.058272 3.452969)) (layer F.SilkS) (width 0.01))
+    (fp_poly (pts (xy -2.671039 -3.071277) (xy -2.648316 -3.048) (xy -2.604899 -2.949922) (xy -2.555194 -2.755791)
+      (xy -2.502812 -2.491647) (xy -2.451365 -2.183531) (xy -2.404467 -1.857484) (xy -2.365728 -1.539546)
+      (xy -2.338761 -1.25576) (xy -2.327179 -1.032164) (xy -2.334593 -0.894801) (xy -2.345821 -0.86728)
+      (xy -2.373383 -0.775801) (xy -2.394425 -0.572165) (xy -2.407957 -0.271094) (xy -2.41299 0.112689)
+      (xy -2.413 0.132816) (xy -2.413 1.065732) (xy -2.256739 1.104951) (xy -2.099422 1.186401)
+      (xy -1.917223 1.338317) (xy -1.749073 1.521363) (xy -1.633903 1.696203) (xy -1.610701 1.757705)
+      (xy -1.593806 1.811924) (xy -1.562155 1.850878) (xy -1.497093 1.87709) (xy -1.379967 1.893085)
+      (xy -1.192124 1.901385) (xy -0.914909 1.904516) (xy -0.529668 1.904999) (xy -0.521992 1.905)
+      (xy -0.114759 1.902905) (xy 0.183846 1.895602) (xy 0.392146 1.881564) (xy 0.52846 1.859264)
+      (xy 0.611108 1.827176) (xy 0.636438 1.808448) (xy 0.6857 1.775472) (xy 0.757921 1.756818)
+      (xy 0.871598 1.753578) (xy 1.045228 1.766846) (xy 1.297308 1.797715) (xy 1.646335 1.847277)
+      (xy 1.879688 1.881907) (xy 2.391353 1.964341) (xy 2.776915 2.040871) (xy 3.036297 2.113236)
+      (xy 3.16942 2.183173) (xy 3.17621 2.252419) (xy 3.056589 2.322714) (xy 2.810479 2.395793)
+      (xy 2.437805 2.473396) (xy 1.93849 2.557259) (xy 1.849209 2.571013) (xy 1.437467 2.632948)
+      (xy 1.133585 2.675607) (xy 0.920057 2.700042) (xy 0.779381 2.707301) (xy 0.694051 2.698435)
+      (xy 0.646564 2.674494) (xy 0.623678 2.644515) (xy 0.58736 2.60553) (xy 0.516578 2.577547)
+      (xy 0.392965 2.558883) (xy 0.198155 2.547855) (xy -0.086219 2.54278) (xy -0.478525 2.541976)
+      (xy -0.495281 2.542007) (xy -1.55575 2.544014) (xy -1.72183 2.817955) (xy -1.951417 3.08259)
+      (xy -2.252272 3.264684) (xy -2.592722 3.354033) (xy -2.941097 3.340433) (xy -3.145408 3.276597)
+      (xy -3.462279 3.077707) (xy -3.687975 2.811529) (xy -3.820931 2.500772) (xy -3.857714 2.184205)
+      (xy -3.539859 2.184205) (xy -3.53524 2.272701) (xy -3.449553 2.572587) (xy -3.276596 2.804518)
+      (xy -3.041561 2.959285) (xy -2.769635 3.027673) (xy -2.48601 3.000472) (xy -2.215875 2.868468)
+      (xy -2.122475 2.789371) (xy -1.922105 2.523765) (xy -1.846304 2.241844) (xy -1.895122 1.952279)
+      (xy -2.068612 1.663742) (xy -2.115545 1.609891) (xy -2.354129 1.429294) (xy -2.619845 1.354376)
+      (xy -2.889391 1.374258) (xy -3.139467 1.47806) (xy -3.346772 1.654904) (xy -3.488003 1.893912)
+      (xy -3.539859 2.184205) (xy -3.857714 2.184205) (xy -3.859581 2.168145) (xy -3.80236 1.836356)
+      (xy -3.647703 1.528114) (xy -3.394043 1.266126) (xy -3.288972 1.194078) (xy -3.051416 1.04775)
+      (xy -3.049708 0.123824) (xy -3.053723 -0.268648) (xy -3.066774 -0.57368) (xy -3.087981 -0.778049)
+      (xy -3.115822 -0.867922) (xy -3.131241 -0.952655) (xy -3.126541 -1.136203) (xy -3.105316 -1.392615)
+      (xy -3.071154 -1.695938) (xy -3.027647 -2.020221) (xy -2.978386 -2.339512) (xy -2.926962 -2.627859)
+      (xy -2.876964 -2.85931) (xy -2.831985 -3.007914) (xy -2.81535 -3.03952) (xy -2.743217 -3.10894)
+      (xy -2.671039 -3.071277)) (layer F.SilkS) (width 0.01))
+    (fp_poly (pts (xy 4.272966 1.925615) (xy 4.251351 2.005902) (xy 4.207305 2.087582) (xy 4.141174 2.223223)
+      (xy 4.14641 2.322657) (xy 4.211722 2.436832) (xy 4.278016 2.55292) (xy 4.267905 2.598318)
+      (xy 4.228492 2.6035) (xy 4.136747 2.550596) (xy 4.09575 2.4765) (xy 4.040555 2.37393)
+      (xy 4.0005 2.3495) (xy 3.939517 2.401834) (xy 3.90525 2.4765) (xy 3.832832 2.579509)
+      (xy 3.769646 2.6035) (xy 3.718847 2.584409) (xy 3.744324 2.510588) (xy 3.802831 2.423067)
+      (xy 3.884251 2.292469) (xy 3.890172 2.201601) (xy 3.832428 2.101461) (xy 3.768135 1.969385)
+      (xy 3.790299 1.916141) (xy 3.873903 1.959964) (xy 3.93371 2.027639) (xy 4.048735 2.18013)
+      (xy 4.092396 2.042565) (xy 4.160804 1.934148) (xy 4.224075 1.905) (xy 4.272966 1.925615)) (layer F.SilkS) (width 0.01))
+    (fp_poly (pts (xy -2.882138 -4.072588) (xy -2.820979 -3.934025) (xy -2.795559 -3.857625) (xy -2.713514 -3.58775)
+      (xy -2.597611 -3.857625) (xy -2.505004 -4.04795) (xy -2.444933 -4.124503) (xy -2.421245 -4.09723)
+      (xy -2.437785 -3.976076) (xy -2.498401 -3.770988) (xy -2.530073 -3.683) (xy -2.637751 -3.419412)
+      (xy -2.718265 -3.274739) (xy -2.770436 -3.250289) (xy -2.793087 -3.347374) (xy -2.794 -3.389496)
+      (xy -2.818563 -3.549217) (xy -2.878744 -3.74239) (xy -2.88925 -3.768456) (xy -2.966047 -3.979024)
+      (xy -2.978047 -4.094325) (xy -2.931052 -4.1275) (xy -2.882138 -4.072588)) (layer F.SilkS) (width 0.01))
+    (fp_poly (pts (xy -2.567194 1.958472) (xy -2.456388 2.084196) (xy -2.413 2.2225) (xy -2.461126 2.368674)
+      (xy -2.574277 2.491791) (xy -2.69875 2.54) (xy -2.810312 2.498363) (xy -2.884715 2.440214)
+      (xy -2.96661 2.307564) (xy -2.9845 2.2225) (xy -2.936375 2.076325) (xy -2.823224 1.953208)
+      (xy -2.69875 1.905) (xy -2.567194 1.958472)) (layer F.SilkS) (width 0.01))
+  )
   (gr_text Burnwire (at 97.7645 97.9865 90) (layer B.SilkS)

Commit message: Places fiducial markers
Parts:
- added REF**: Fiducial_0.5mm_Dia_1mm_Outer, Fiducials:Fiducial_0.5mm_Dia_1mm_Outer, F.Cu at (69.2, 105.7)
- added REF**: Fiducial_0.5mm_Dia_1mm_Outer, Fiducials:Fiducial_0.5mm_Dia_1mm_Outer, F.Cu at (121.9, 108.1)
- added REF**: Fiducial_0.5mm_Dia_1mm_Outer, Fiducials:Fiducial_0.5mm_Dia_1mm_Outer, B.Cu at (58.6, 44.0)
- added REF**: Fiducial_0.5mm_Dia_1mm_Outer, Fiducials:Fiducial_0.5mm_Dia_1mm_Outer, B.Cu at (129.1, 42.7)
Changed lines of the file:
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@@
-(kicad_pcb (version 4) (host pcbnew 4.0.6)
+(kicad_pcb (version 4) (host pcbnew 4.0.7)
   (general
     (links 0)
@@
     (tracks 2134)
     (zones 0)
-    (modules 407)
+    (modules 411)
     (nets 175)
   )
@@
       (xy -2.69875 1.905) (xy -2.567194 1.958472)) (layer F.SilkS) (width 0.01))
   )
+  (module Fiducials:Fiducial_0.5mm_Dia_1mm_Outer (layer F.Cu)
+    (at 69.1645 105.7065)
+    (descr "Circular Fiducial, 0.5mm bare copper top; 1mm keepout (Level C)")
+    (tags marker)
+    (attr virtual)
+    (fp_text reference REF** (at 0 -1.5) (layer F.SilkS)
+      (effects (font (size 1 1) (thickness 0.15)))
+    )
+    (fp_text value Fiducial_0.5mm_Dia_1mm_Outer (at 0 1.5) (layer F.Fab)
+      (effects (font (size 1 1) (thickness 0.15)))
+    )
+    (fp_circle (center 0 0) (end 0.5 0) (layer F.Fab) (width 0.1))
+    (fp_text user %R (at 0 0) (layer F.Fab)
+      (effects (font (size 0.2 0.2) (thickness 0.04)))
+    )
+    (fp_circle (center 0 0) (end 0.75 0) (layer F.CrtYd) (width 0.05))
+    (pad ~ smd circle (at 0 0) (size 0.5 0.5) (layers F.Cu F.Mask)
+      (solder_mask_margin 0.25) (clearance 0.25))
+  )
+  (module Fiducials:Fiducial_0.5mm_Dia_1mm_Outer (layer F.Cu)
+    (at 121.8695 108.1195)
+    (descr "Circular Fiducial, 0.5mm bare copper top; 1mm keepout (Level C)")
+    (tags marker)
+    (attr virtual)
+    (fp_text reference REF** (at 0 -1.5) (layer F.SilkS)
+      (effects (font (size 1 1) (thickness 0.15)))
+    )
+    (fp_text value Fiducial_0.5mm_Dia_1mm_Outer (at 0 1.5) (layer F.Fab)
+      (effects (font (size 1 1) (thickness 0.15)))
+    )
+    (fp_circle (center 0 0) (end 0.5 0) (layer F.Fab) (width 0.1))
+    (fp_text user %R (at 0 0) (layer F.Fab)
+      (effects (font (size 0.2 0.2) (thickness 0.04)))
+    )
+    (fp_circle (center 0 0) (end 0.75 0) (layer F.CrtYd) (width 0.05))
+    (pad ~ smd circle (at 0 0) (size 0.5 0.5) (layers F.Cu F.Mask)
+      (solder_mask_margin 0.25) (clearance 0.25))
+  )
+  (module Fiducials:Fiducial_0.5mm_Dia_1mm_Outer (layer B.Cu)
+    (at 58.6235 43.9845)
+    (descr "Circular Fiducial, 0.5mm bare copper top; 1mm keepout (Level C)")
+    (tags marker)
+    (attr virtual)
+    (fp_text reference REF** (at 0 1.5) (layer B.SilkS)
+      (effects (font (size 1 1) (thickness 0.15)) (justify mirror))
+    )
+    (fp_text value Fiducial_0.5mm_Dia_1mm_Outer (at 0 -1.5) (layer B.Fab)
+      (effects (font (size 1 1) (thickness 0.15)) (justify mirror))
+    )
+    (fp_circle (center 0 0) (end 0.5 0) (layer B.Fab) (width 0.1))
+    (fp_text user %R (at 0 0) (layer B.Fab)
+      (effects (font (size 0.2 0.2) (thickness 0.04)) (justify mirror))
+    )
+    (fp_circle (center 0 0) (end 0.75 0) (layer B.CrtYd) (width 0.05))
+    (pad ~ smd circle (at 0 0) (size 0.5 0.5) (layers B.Cu B.Mask)
+      (solder_mask_margin 0.25) (clearance 0.25))
+  )
+  (module Fiducials:Fiducial_0.5mm_Dia_1mm_Outer (layer B.Cu)
+    (at 129.1085 42.7145)
+    (descr "Circular Fiducial, 0.5mm bare copper top; 1mm keepout (Level C)")
+    (tags marker)
+    (attr virtual)
+    (fp_text reference REF** (at 0 1.5) (layer B.SilkS)
+      (effects (font (size 1 1) (thickness 0.15)) (justify mirror))
+    )
+    (fp_text value Fiducial_0.5mm_Dia_1mm_Outer (at 0 -1.5) (layer B.Fab)
+      (effects (font (size 1 1) (thickness 0.15)) (justify mirror))
+    )
+    (fp_circle (center 0 0) (end 0.5 0) (layer B.Fab) (width 0.1))
+    (fp_text user %R (at 0 0) (layer B.Fab)
+      (effects (font (size 0.2 0.2) (thickness 0.04)) (justify mirror))
+    )
+    (fp_circle (center 0 0) (end 0.75 0) (layer B.CrtYd) (width 0.05))
+    (pad ~ smd circle (at 0 0) (size 0.5 0.5) (layers B.Cu B.Mask)
+      (solder_mask_margin 0.25) (clearance 0.25))
+  )
   (gr_text Burnwire (at 97.7645 97.9865 90) (layer B.SilkS)

Commit message: Auto stash before merge of "master" and "origin/master"
Parts:
- removed the REF** at (69.2, 105.7)
- removed the REF** at (121.9, 108.1)
- removed the REF** at (58.6, 44.0)
- removed the REF** at (129.1, 42.7)
- added FID1: Fiducial, Fiducials:Fiducial_0.5mm_Dia_1mm_Outer, F.Cu at (69.8, 107.6)
- added FID2: Fiducial, Fiducials:Fiducial_0.5mm_Dia_1mm_Outer, F.Cu at (121.9, 108.5)
- added FID3: Fiducial, Fiducials:Fiducial_0.5mm_Dia_1mm_Outer, F.Cu at (96.2, 40.3)
- added FID4: Fiducial, Fiducials:Fiducial_0.5mm_Dia_1mm_Outer, B.Cu at (91.9, 114.5)
- added FID5: Fiducial, Fiducials:Fiducial_0.5mm_Dia_1mm_Outer, B.Cu at (59.0, 48.8)
- added FID6: Fiducial, Fiducials:Fiducial_0.5mm_Dia_1mm_Outer, B.Cu at (127.8, 43.0)
Connections:
- U1 pad 9: (no net) -> Net-(U1-Pad9)
- U10 pad 14: (no net) -> Net-(U10-Pad14)
- U10 pad 15: (no net) -> Net-(U10-Pad15)
- U10 pad 16: (no net) -> Net-(U10-Pad16)
- U3 pad 1: (no net) -> Net-(U3-Pad1)
- U3 pad 14: (no net) -> Net-(U3-Pad14)
- U3 pad 17: (no net) -> Net-(U3-Pad17)
- U3 pad 18: (no net) -> Net-(U3-Pad18)
- U3 pad 19: (no net) -> Net-(U3-Pad19)
- U3 pad 26: (no net) -> Net-(U3-Pad26)
- U3 pad 27: (no net) -> Net-(U3-Pad27)
- U3 pad 28: (no net) -> Net-(U3-Pad28)
- U3 pad 30: (no net) -> Net-(U3-Pad30)
- U3 pad 31: (no net) -> Net-(U3-Pad31)
- U3 pad 32: (no net) -> Net-(U3-Pad32)
- U3 pad 33: (no net) -> Net-(U3-Pad33)
- U3 pad 34: (no net) -> Net-(U3-Pad34)
- U3 pad 35: (no net) -> Net-(U3-Pad35)
- U3 pad 36: (no net) -> Net-(U3-Pad36)
- U3 pad 37: (no net) -> Net-(U3-Pad37)
- U3 pad 38: (no net) -> Net-(U3-Pad38)
- U3 pad 39: (no net) -> Net-(U3-Pad39)
- U3 pad 40: (no net) -> Net-(U3-Pad40)
- U3 pad 41: (no net) -> Net-(U3-Pad41)
- U3 pad 42: (no net) -> Net-(U3-Pad42)
- U3 pad 43: (no net) -> Net-(U3-Pad43)
- U3 pad 44: (no net) -> Net-(U3-Pad44)
- U3 pad 45: (no net) -> Net-(U3-Pad45)
- U3 pad 46: (no net) -> Net-(U3-Pad46)
- U3 pad 47: (no net) -> Net-(U3-Pad47)
- U3 pad 48: (no net) -> Net-(U3-Pad48)
- U3 pad 49: (no net) -> Net-(U3-Pad49)
- U3 pad 50: (no net) -> Net-(U3-Pad50)
- U3 pad 51: (no net) -> Net-(U3-Pad51)
- U3 pad 62: (no net) -> Net-(U3-Pad62)
- U3 pad 7: (no net) -> Net-(U3-Pad7)
- U3 pad 8: (no net) -> Net-(U3-Pad8)
- U3 pad 9: (no net) -> Net-(U3-Pad9)
- U5 pad 14: (no net) -> Net-(U5-Pad14)
- U5 pad 15: (no net) -> Net-(U5-Pad15)
- U5 pad 16: (no net) -> Net-(U5-Pad16)
- U6 pad 9: (no net) -> Net-(U6-Pad9)
- U8 pad 1: (no net) -> Net-(U8-Pad1)
- U8 pad 14: (no net) -> Net-(U8-Pad14)
- U8 pad 17: (no net) -> Net-(U8-Pad17)
- U8 pad 18: (no net) -> Net-(U8-Pad18)
- U8 pad 19: (no net) -> Net-(U8-Pad19)
- U8 pad 26: (no net) -> Net-(U8-Pad26)
- U8 pad 27: (no net) -> Net-(U8-Pad27)
- U8 pad 28: (no net) -> Net-(U8-Pad28)
- U8 pad 30: (no net) -> Net-(U8-Pad30)
- U8 pad 31: (no net) -> Net-(U8-Pad31)
- U8 pad 32: (no net) -> Net-(U8-Pad32)
- U8 pad 33: (no net) -> Net-(U8-Pad33)
- U8 pad 34: (no net) -> Net-(U8-Pad34)
- U8 pad 35: (no net) -> Net-(U8-Pad35)
- U8 pad 36: (no net) -> Net-(U8-Pad36)
- U8 pad 37: (no net) -> Net-(U8-Pad37)
- U8 pad 38: (no net) -> Net-(U8-Pad38)
- U8 pad 39: (no net) -> Net-(U8-Pad39)
- U8 pad 40: (no net) -> Net-(U8-Pad40)
- U8 pad 41: (no net) -> Net-(U8-Pad41)
- U8 pad 42: (no net) -> Net-(U8-Pad42)
- U8 pad 43: (no net) -> Net-(U8-Pad43)
- U8 pad 44: (no net) -> Net-(U8-Pad44)
- U8 pad 45: (no net) -> Net-(U8-Pad45)
- U8 pad 46: (no net) -> Net-(U8-Pad46)
- U8 pad 47: (no net) -> Net-(U8-Pad47)
- U8 pad 48: (no net) -> Net-(U8-Pad48)
- U8 pad 49: (no net) -> Net-(U8-Pad49)
- U8 pad 50: (no net) -> Net-(U8-Pad50)
- U8 pad 51: (no net) -> Net-(U8-Pad51)
- U8 pad 62: (no net) -> Net-(U8-Pad62)
- U8 pad 7: (no net) -> Net-(U8-Pad7)
- U8 pad 8: (no net) -> Net-(U8-Pad8)
- U8 pad 9: (no net) -> Net-(U8-Pad9)
